File: IOC Single/IOC_Single.kicad_sch (KiCad schematic)
At the start: 6 parts, among them J1 ICSP, SW1 SW_DIP_x08, U1 PIC18F47Q43-E/P

Commit message: Code and hardware working
Connections:
- net at SW1.10: now also U1.44 (RC6); no longer U1.4 (RD6)
- net at SW1.11: now also U1.43 (RC5); no longer U1.3 (RD5)
- net at SW1.12: now also U1.42 (RC4); no longer U1.2 (RD4)
- net at SW1.13: now also U1.37 (RC3); no longer U1.41 (RD3)
- net at SW1.14: now also U1.36 (RC2); no longer U1.40 (RD2)
- net at SW1.15: now also U1.35 (RC1); no longer U1.39 (RD1)
- net at SW1.16: now also U1.32 (RC0); no longer U1.38 (RD0)
- net at SW1.9: now also U1.1 (RC7); no longer U1.5 (RD7)
- net at BAR1.13 (K): now also U1.5 (RD7); no longer U1.1 (RC7)
- net at BAR1.14 (K): now also U1.4 (RD6); no longer U1.44 (RC6)
- net at BAR1.15 (K): now also U1.3 (RD5); no longer U1.43 (RC5)
- net at BAR1.16 (K): now also U1.2 (RD4); no longer U1.42 (RC4)
- net at BAR1.17 (K): now also U1.41 (RD3); no longer U1.37 (RC3)
- net at BAR1.18 (K): now also U1.40 (RD2); no longer U1.36 (RC2)
- net at BAR1.19 (K): now also U1.39 (RD1); no longer U1.35 (RC1)
- net at BAR1.20 (K): now also U1.38 (RD0); no longer U1.32 (RC0)
Other:
- moved on the sheet: BAR1, RN1, SW1

Commit message: updated schematic and saved as PDF
Other:
- note added: "Note, the device shown is the TQFP-44 packaged variant. The pin assignments vary from one package type to another."
- company: (none) -> Dewayne Hafenstein
- title: (none) -> IOC Non-Vectored Interrupts
Changed lines of the file:
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@@
 	(generator_version "9.0")
 	(paper "A")
+	(title_block
+		(title "IOC Non-Vectored Interrupts")
+		(date "2026-04-10")
+		(rev "1")
+		(company "Dewayne Hafenstein")
+		(comment 1 "Interrupt On Change")
+	)
+	(text "Note, the device shown is the TQFP-44 \npackaged variant. The pin assignments\nvary from one package type to another."
+		(exclude_from_sim no)
+		(at 131.064 132.842 0)
+		(effects
+			(font
+				(size 1.27 1.27)
+			)
+		)
+	)
 	(junction
 		(at 80.01 116.84)
