File: IOC Vectored/IOC_Vectored.kicad_sch (KiCad schematic)
At the start: 6 parts, among them J1 ICSP, SW1 SW_DIP_x08, U1 PIC18F47Q43-I/PT

Commit message: Updated Documentation
Other:
- title: IOC Non-Vectored Interrupts -> IOC Vectored Interrupts
Changed lines of the file:
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@@
 	(paper "A")
 	(title_block
-		(title "IOC Non-Vectored Interrupts")
+		(title "IOC Vectored Interrupts")
 		(date "2026-04-10")
 		(rev "1")
