File: 01 UART/UART 02 DMA TX Stream/UART 02 DMA TX Stream.kicad_sch (KiCad schematic)
At the start: 15 parts, among them J101 ICSP, J102 USB_A, U101 PIC18F47Q43-I/PT, U103 FT232RL

Commit message: Revisions to order
Co-authored-by: Copilot <copilot@github.com>
Other:
- note removed: "NOTE: A common mistake is to wire the controllers TX output to the TX pin of the FT232. The FT232 is labeled from the perspective of a remote device you want to connect to, so the FT232 TX pin should be connected to the controllers RX input, FT232 RX pin to the controllers TX output, etc. This is NOT the case when using an RS232 level shifter such as the MAX232, which is simply translating the si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"
- note removed: "Notes: 1. Implement one or the other interface options, USB or RS-232, but not both. 2. Place C101 and C102 physically close to U101. 3. For USB interface, place C109 and C110 physically close to U103. 4. For RS-232 interface, locate C103 - C107 physically close to U102. 5. This example does not use hardware or software flow control!"
Changed lines of the file:
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@@
 		(company "Dewayne Hafenstein")
-	)
-	(text "NOTE:  A common mistake is to wire the controllers TX output to the TX\npin of the FT232.  The  FT232 is labeled from the perspective of a remote\ndevice you want to connect to, so the FT232 TX pin should be connected to\nthe controllers RX input, FT232 RX pin to the controllers TX output, etc. \n\nThis is NOT the case when using an RS232 level shifter such as the \nMAX232, which is simply translating the signals to RS-232 levels. "
-		(exclude_from_sim no)
-		(at 63.246 187.96 0)
-		(effects
-			(font
-				(size 1.27 1.27)
-			)
-			(justify left)
-		)
-	)
-	(text "Notes:\n1. Implement one or the other interface options, USB or RS-232,\n   but not both.\n2. Place C101 and C102 physically close to U101.\n3. For USB interface, place C109 and C110 physically close to U103.\n4. For RS-232 interface, locate C103 - C107 physically close to U102.\n5. This example does not use hardware or software flow control!"
-		(exclude_from_sim no)
-		(at 30.734 158.242 0)
-		(effects
-			(font
-				(size 1.27 1.27)
-			)
-			(justify left)
-		)
 	)
 	(text "USB Interface"
