File: 05 CRC/CRC 01 Stream Verify/CRC 01 Stream Verify.kicad_sch (KiCad schematic)
At the start: 22 parts, among them J101 ICSP, J102 USB_A, J103 DB9_Pins, U101 PIC18F47Q43-I/PT, U102 MAX232, U103 FT232RL

Commit message: Added more examples
Co-authored-by: Copilot <copilot@github.com>
Other:
- title: 03 UART DMA RX Buffer -> CRC 01 Stream Verify
Changed lines of the file:
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@@
 	(paper "A")
 	(title_block
-		(title "03 UART DMA RX Buffer")
+		(title "CRC 01 Stream Verify")
 		(date "2026-04-11")
 		(rev "1")
@@
 		)
 		(instances
-			(project "UART 03 DMA RX Buffer"
+			(project "CRC 01 Stream Verify"
 				(path "/d3b5dd27-4845-413f-badb-7f64f7fb8d77"
 					(reference "D102")
@@
 		)
 		(instances
-			(project "UART 03 DMA RX Buffer"
+			(project "CRC 01 Stream Verify"
 				(path "/d3b5dd27-4845-413f-badb-7f64f7fb8d77"
 					(reference "#PWR0117")
@@
 		)
 		(instances
-			(project "UART 03 DMA RX Buffer"
+			(project "CRC 01 Stream Verify"
 				(path "/d3b5dd27-4845-413f-badb-7f64f7fb8d77"
 					(reference "#PWR0106")
@@
 		)
 		(instances
-			(project "UART 03 DMA RX Buffer"
+			(project "CRC 01 Stream Verify"
 				(path "/d3b5dd27-4845-413f-badb-7f64f7fb8d77"
 					(reference "#PWR0112")
@@
 		)
 		(instances
-			(project "UART 03 DMA RX Buffer"
+			(project "CRC 01 Stream Verify"
 				(path "/d3b5dd27-4845-413f-badb-7f64f7fb8d77"
 					(reference "C102")
@@
 		)
 		(instances
-			(project "UART 03 DMA RX Buffer"
+			(project "CRC 01 Stream Verify"
 				(path "/d3b5dd27-4845-413f-badb-7f64f7fb8d77"
 					(reference "#PWR0101")
@@
 		)
 		(instances
-			(project "UART 03 DMA RX Buffer"
+			(project "CRC 01 Stream Verify"
 				(path "/d3b5dd27-4845-413f-badb-7f64f7fb8d77"
 					(reference "#PWR0116")
@@
 		)
 		(instances
-			(project "UART 03 DMA RX Buffer"
+			(project "CRC 01 Stream Verify"
 				(path "/d3b5dd27-4845-413f-badb-7f64f7fb8d77"
 					(reference "#PWR0114")
@@
 		)
 		(instances
-			(project "UART 03 DMA RX Buffer"
+			(project "CRC 01 Stream Verify"
 				(path "/d3b5dd27-4845-413f-badb-7f64f7fb8d77"
 					(reference "J101")
@@
 		)
 		(instances
-			(project "UART 03 DMA RX Buffer"
+			(project "CRC 01 Stream Verify"
 				(path "/d3b5dd27-4845-413f-badb-7f64f7fb8d77"
 					(reference "#PWR0102")
@@
 		)
 		(instances
-			(project "UART 03 DMA RX Buffer"
+			(project "CRC 01 Stream Verify"
 				(path "/d3b5dd27-4845-413f-badb-7f64f7fb8d77"
 					(reference "#PWR0103")
@@
 		)
 		(instances
-			(project "UART 03 DMA RX Buffer"
+			(project "CRC 01 Stream Verify"
 				(path "/d3b5dd27-4845-413f-badb-7f64f7fb8d77"
 					(reference "C103")
@@
 		)
 		(instances
-			(project "UART 03 DMA RX Buffer"
+			(project "CRC 01 Stream Verify"
 				(path "/d3b5dd27-4845-413f-badb-7f64f7fb8d77"
 					(reference "J103")
@@
 		)
 		(instances
-			(project "UART 03 DMA RX Buffer"
+			(project "CRC 01 Stream Verify"
 				(path "/d3b5dd27-4845-413f-badb-7f64f7fb8d77"
 					(reference "#PWR0108")
@@
 		)
 		(instances
-			(project "UART 03 DMA RX Buffer"
+			(project "CRC 01 Stream Verify"
 				(path "/d3b5dd27-4845-413f-badb-7f64f7fb8d77"
 					(reference "#PWR0109")
@@
 		)
 		(instances
-			(project "UART 03 DMA RX Buffer"
+			(project "CRC 01 Stream Verify"
 				(path "/d3b5dd27-4845-413f-badb-7f64f7fb8d77"
 					(reference "#PWR0107")
@@
 		)
 		(instances
-			(project "UART 03 DMA RX Buffer"
+			(project "CRC 01 Stream Verify"
 				(path "/d3b5dd27-4845-413f-badb-7f64f7fb8d77"
 					(reference "R103")
@@
 		)
 		(instances
-			(project "UART 03 DMA RX Buffer"
+			(project "CRC 01 Stream Verify"
 				(path "/d3b5dd27-4845-413f-badb-7f64f7fb8d77"
 					(reference "D101")
@@
 		)
 		(instances
-			(project "UART 03 DMA RX Buffer"
+			(project "CRC 01 Stream Verify"
 				(path "/d3b5dd27-4845-413f-badb-7f64f7fb8d77"
 					(reference "C101")
@@
 		)
 		(instances
-			(project "UART 03 DMA RX Buffer"
+			(project "CRC 01 Stream Verify"
 				(path "/d3b5dd27-4845-413f-badb-7f64f7fb8d77"
 					(reference "C108")
@@
 		)
 		(instances
-			(project "UART 03 DMA RX Buffer"
+			(project "CRC 01 Stream Verify"
 				(path "/d3b5dd27-4845-413f-badb-7f64f7fb8d77"
 					(reference "C107")
@@
 		)
 		(instances
-			(project "UART 03 DMA RX Buffer"
+			(project "CRC 01 Stream Verify"
 				(path "/d3b5dd27-4845-413f-badb-7f64f7fb8d77"
 					(reference "#PWR0110")
@@
 		)
 		(instances
-			(project "UART 03 DMA RX Buffer"
+			(project "CRC 01 Stream Verify"
 				(path "/d3b5dd27-4845-413f-badb-7f64f7fb8d77"
 					(reference "#PWR0105")
@@
 		)
 		(instances
-			(project "UART 03 DMA RX Buffer"
+			(project "CRC 01 Stream Verify"
 				(path "/d3b5dd27-4845-413f-badb-7f64f7fb8d77"
 					(reference "R101")
@@
 		)
 		(instances
-			(project "UART 03 DMA RX Buffer"
+			(project "CRC 01 Stream Verify"
 				(path "/d3b5dd27-4845-413f-badb-7f64f7fb8d77"
 					(reference "R104")
@@
 		)
 		(instances
-			(project "UART 03 DMA RX Buffer"
+			(project "CRC 01 Stream Verify"
 				(path "/d3b5dd27-4845-413f-badb-7f64f7fb8d77"
 					(reference "#PWR0115")
@@
 		)
 		(instances
-			(project "UART 03 DMA RX Buffer"
+			(project "CRC 01 Stream Verify"
 				(path "/d3b5dd27-4845-413f-badb-7f64f7fb8d77"
 					(reference "#PWR0111")
@@
 		)
 		(instances
-			(project "UART 03 DMA RX Buffer"
+			(project "CRC 01 Stream Verify"
 				(path "/d3b5dd27-4845-413f-badb-7f64f7fb8d77"
 					(reference "J102")
@@
 		)
 		(instances
-			(project "UART 03 DMA RX Buffer"
+			(project "CRC 01 Stream Verify"
 				(path "/d3b5dd27-4845-413f-badb-7f64f7fb8d77"
 					(reference "U102")
@@
 		)
 		(instances
-			(project "UART 03 DMA RX Buffer"
+			(project "CRC 01 Stream Verify"
 				(path "/d3b5dd27-4845-413f-badb-7f64f7fb8d77"
 					(reference "C104")
@@
 		)
 		(instances
-			(project "UART 03 DMA RX Buffer"
+			(project "CRC 01 Stream Verify"
 				(path "/d3b5dd27-4845-413f-badb-7f64f7fb8d77"
 					(reference "C106")
@@
 		)
 		(instances
-			(project "UART 03 DMA RX Buffer"
+			(project "CRC 01 Stream Verify"
 				(path "/d3b5dd27-4845-413f-badb-7f64f7fb8d77"
 					(reference "U101")
@@
 		)
 		(instances
-			(project "UART 03 DMA RX Buffer"
+			(project "CRC 01 Stream Verify"
 				(path "/d3b5dd27-4845-413f-badb-7f64f7fb8d77"
 					(reference "#PWR0104")
@@
 		)
 		(instances
-			(project "UART 03 DMA RX Buffer"
+			(project "CRC 01 Stream Verify"
 				(path "/d3b5dd27-4845-413f-badb-7f64f7fb8d77"
 					(reference "C110")
@@
 		)
 		(instances
-			(project "UART 03 DMA RX Buffer"
+			(project "CRC 01 Stream Verify"
 				(path "/d3b5dd27-4845-413f-badb-7f64f7fb8d77"
 					(reference "C109")
@@
 		)
 		(instances
-			(project "UART 03 DMA RX Buffer"
+			(project "CRC 01 Stream Verify"
 				(path "/d3b5dd27-4845-413f-badb-7f64f7fb8d77"
 					(reference "U103")
@@
 		)
 		(instances
-			(project "UART 03 DMA RX Buffer"
+			(project "CRC 01 Stream Verify"
 				(path "/d3b5dd27-4845-413f-badb-7f64f7fb8d77"
 					(reference "R102")
@@
 		)
 		(instances
-			(project "UART 03 DMA RX Buffer"
+			(project "CRC 01 Stream Verify"
 				(path "/d3b5dd27-4845-413f-badb-7f64f7fb8d77"
 					(reference "#PWR0113")
@@
 		)
 		(instances
-			(project "UART 03 DMA RX Buffer"
+			(project "CRC 01 Stream Verify"
 				(path "/d3b5dd27-4845-413f-badb-7f64f7fb8d77"
 					(reference "C105")
