File: 05 CRC/CRC 01 Stream Verify/CRC 01 Stream Verify.kicad_sch (KiCad schematic)
At the start: 22 parts, among them J101 ICSP, J102 USB_A, J103 DB9_Pins, U101 PIC18F47Q43-I/PT, U102 MAX232, U103 FT232RL

Commit message: cleanup
Connections:
- removed net CTS: U101.11 (RB3), U102.10 (T2IN), U103.3 (RTS)
- net Clear_to_Send: no longer names the net of J103.8
- net Clear_to_Send: no longer U102.7 (T2OUT)
- removed net RTS: U101.10 (RB2), U102.9 (R2OUT), U103.11 (CTS)
- net Request_to_Send: no longer names the net of J103.7
- net Request_to_Send: no longer U102.8 (R2IN)
- no-connect marks 40 -> 48
Changed lines of the file:
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@@
+	)
+	(no_connect
+		(at 60.96 90.17)
 	)
 	(no_connect
@@
 	)
 	(no_connect
+		(at 161.29 64.77)
+	)
+	(no_connect
 		(at 232.41 69.85)
 	)
@@
 	)
 	(no_connect
+		(at 162.56 121.92)
+	)
+	(no_connect
 		(at 162.56 129.54)
 	)
@@
 	)
 	(no_connect
+		(at 161.29 74.93)
+	)
+	(no_connect
 		(at 60.96 59.69)
 	)
@@
 	)
 	(no_connect
+		(at 232.41 59.69)
+	)
+	(no_connect
 		(at 104.14 97.79)
 	)
@@
 	)
 	(no_connect
+		(at 232.41 64.77)
+	)
+	(no_connect
 		(at 60.96 120.65)
 	)
@@
 	)
 	(no_connect
+		(at 60.96 87.63)
+	)
+	(no_connect
 		(at 104.14 110.49)
 	)
 	(no_connect
 		(at 60.96 92.71)
+	)
+	(no_connect
+		(at 162.56 119.38)
 	)
 	(bus_entry
@@
 	)
 	(bus_entry
-		(at 30.48 85.09)
-		(size 2.54 2.54)
-		(stroke
-			(width 0)
-			(type default)
-		)
-	)
-	(bus_entry
 		(at 137.16 67.31)
 		(size 2.54 2.54)
@@
 	)
 	(bus_entry
-		(at 137.16 62.23)
-		(size 2.54 2.54)
-		(stroke
-			(width 0)
-			(type default)
-		)
-	)
-	(bus_entry
-		(at 137.16 116.84)
-		(size 2.54 2.54)
-		(stroke
-			(width 0)
-			(type default)
-		)
-	)
-	(bus_entry
-		(at 137.16 119.38)
-		(size 2.54 2.54)
-		(stroke
-			(width 0)
-			(type default)
-		)
-	)
-	(bus_entry
 		(at 137.16 111.76)
-		(size 2.54 2.54)
-		(stroke
-			(width 0)
-			(type default)
-		)
-	)
-	(bus_entry
-		(at 137.16 72.39)
-		(size 2.54 2.54)
-		(stroke
-			(width 0)
-			(type default)
-		)
-	)
-	(bus_entry
-		(at 30.48 87.63)
 		(size 2.54 2.54)
 		(stroke
@@
 	(wire
 		(pts
-			(xy 228.6 59.69) (xy 232.41 59.69)
-		)
-		(stroke
-			(width 0)
-			(type default)
-		)
-	)
-	(wire
-		(pts
 			(xy 234.95 146.05) (xy 234.95 147.32)
 		)
@@
 	(wire
 		(pts
-			(xy 139.7 121.92) (xy 162.56 121.92)
-		)
-		(stroke
-			(width 0)
-			(type default)
-		)
-	)
-	(wire
-		(pts
 			(xy 185.42 104.14) (xy 180.34 104.14)
 		)
@@
 	(wire
 		(pts
-			(xy 231.14 54.61) (xy 232.41 54.61)
+			(xy 228.6 54.61) (xy 232.41 54.61)
 		)
 		(stroke
@@
 	(wire
 		(pts
-			(xy 139.7 64.77) (xy 161.29 64.77)
-		)
-		(stroke
-			(width 0)
-			(type default)
-		)
-	)
-	(wire
-		(pts
 			(xy 205.74 34.29) (xy 201.93 34.29)
 		)
@@
 	(wire
 		(pts
-			(xy 232.41 67.31) (xy 231.14 67.31)
+			(xy 232.41 67.31) (xy 228.6 67.31)
 		)
 		(stroke
@@
 	(wire
 		(pts
-			(xy 201.93 74.93) (xy 228.6 74.93)
-		)
-		(stroke
-			(width 0)
-			(type default)
-		)
-	)
-	(wire
-		(pts
 			(xy 177.8 157.48) (xy 177.8 160.02)
 		)
@@
 	(wire
 		(pts
-			(xy 201.93 64.77) (xy 232.41 64.77)
-		)
-		(stroke
-			(width 0)
-			(type default)
-		)
-	)
-	(wire
-		(pts
 			(xy 205.74 41.91) (xy 201.93 41.91)
 		)
@@
 	(wire
 		(pts
-			(xy 33.02 90.17) (xy 60.96 90.17)
-		)
-		(stroke
-			(width 0)
-			(type default)
-		)
-	)
-	(wire
-		(pts
 			(xy 114.3 52.07) (xy 114.3 53.34)
 		)
@@
 		)
 	)
-	(wire
-		(pts
-			(xy 33.02 87.63) (xy 60.96 87.63)
-		)
-		(stroke
-			(width 0)
-			(type default)
-		)
-	)
 	(bus
 		(pts
@@
 	(wire
 		(pts
-			(xy 139.7 119.38) (xy 162.56 119.38)
-		)
-		(stroke
-			(width 0)
-			(type default)
-		)
-	)
-	(wire
-		(pts
 			(xy 104.14 54.61) (xy 106.68 54.61)
 		)
@@
 	(wire
 		(pts
-			(xy 139.7 74.93) (xy 161.29 74.93)
-		)
-		(stroke
-			(width 0)
-			(type default)
-		)
-	)
-	(wire
-		(pts
 			(xy 140.97 142.24) (xy 143.51 142.24)
 		)
@@
 	(wire
 		(pts
-			(xy 228.6 74.93) (xy 228.6 59.69)
-		)
-		(stroke
-			(width 0)
-			(type default)
-		)
-	)
-	(wire
-		(pts
 			(xy 238.76 132.08) (xy 238.76 134.62)
 		)
@@
 	(wire
 		(pts
-			(xy 231.14 67.31) (xy 231.14 54.61)
+			(xy 228.6 67.31) (xy 228.6 54.61)
 		)
 		(stroke
@@
 		)
 	)
-	(label "Request_to_Send"
-		(at 203.2 74.93 0)
-		(effects
-			(font
-				(size 1.27 1.27)
-			)
-			(justify left bottom)
-		)
-	)
 	(label "UART1_TX"
 		(at 33.02 82.55 0)
@@
 		)
 	)
-	(label "RTS"
-		(at 33.02 87.63 0)
-		(effects
-			(font
-				(size 1.27 1.27)
-			)
-			(justify left bottom)
-		)
-	)
-	(label "RTS"
-		(at 140.97 74.93 0)
-		(effects
-			(font
-				(size 1.27 1.27)
-			)
-			(justify left bottom)
-		)
-	)
 	(label "TxD"
 		(at 203.2 59.69 0)
@@
 		)
 	)
-	(label "Clear_to_Send"
-		(at 203.2 64.77 0)
-		(effects
-			(font
-				(size 1.27 1.27)
-			)
-			(justify left bottom)
-		)
-	)
-	(label "CTS"
-		(at 33.02 90.17 0)
-		(effects
-			(font
-				(size 1.27 1.27)
-			)
-			(justify left bottom)
-		)
-	)
 	(label "RxD"
 		(at 203.2 69.85 0)
@@
 		(effects
 			(font
-				(size 1.27 1.27)
-			)
-			(justify left bottom)
-		)
-	)
-	(label "CTS"
-		(at 140.97 64.77 0)
-		(effects
-			(font
-				(size 1.27 1.27)
-			)
-			(justify left bottom)
-		)
-	)
-	(label "RTS"
-		(at 139.7 121.92 0)
-		(effects
-			(font
-				(size 1.27 1.27)
-			)
-			(justify left bottom)
-		)
-	)
-	(label "CTS"
-		(at 139.7 119.38 0)
-		(effects
-			(font
