File: 06 FVR/FVR 01 Reference Bring Up/FVR 01 Reference Bring Up.kicad_sch (KiCad schematic)
At the start: 22 parts, among them J101 ICSP, J102 USB_A, J103 DB9_Pins, U101 PIC18F47Q43-I/PT, U102 MAX232, U103 FT232RL

Commit message: Added more examples
Co-authored-by: Copilot <copilot@github.com>
Parts:
- added D103: Enabled, symbol Device:LED_Small
- added R105: 270, symbol Device:R_US
- J103: value DB9_Pins -> DE9_Pins
Connections:
- net +5V: now also R105.1
- removed net CTS: U101.11 (RB3), U102.10 (T2IN), U103.3 (RTS)
- net Clear_to_Send: no longer names the net of U102.7 (T2OUT)
- net Clear_to_Send: no longer J103.8
- removed net RTS: U101.10 (RB2), U102.9 (R2OUT), U103.11 (CTS)
- net Request_to_Send: no longer names the net of U102.8 (R2IN)
- net Request_to_Send: no longer J103.7
- new net: D103.2 (A), R105.2
- new net: D103.1 (K), U101.10 (RB2)
- new net: J103.7, J103.8
- no-connect marks 40 -> 47
Other:
- note added: "NOTE: A common mistake is to wire the controllers TX output to the TX pin of the FT232. The FT232 is labeled from the perspective of a remote device you want to connect to, so the FT232 TX pin should be connected to the controllers RX input, FT232 RX pin to the controllers TX output, etc. This is NOT the case when using an RS232 level shifter such as the MAX232, which is simply translating the si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"
- note added: "Notes: 1. Implement one or the other interface options, USB or RS-232, but not both. 2. Place C101 and C102 physically close to U101. 3. For USB interface, place C109 and C110 physically close to U103. 4. For RS-232 interface, locate C103 - C107 physically close to U102. 5. This example does not use hardware or software flow control!"
- note removed: "NOTE: A common mistake is to wire the controllers TX output to the TX pin of the FT232. The FT232 is labeled from the perspective of a remote device you want to connect to, so the FT232 TX pin should be connected to the controllers RX input, FT232 RX pin to the controllers TX output, etc. Cross connect RTS and CTS as well. This is NOT the case when using an RS232 level shifter such as the MAX232,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"
- note removed: "Notes: 1. Implement one or the other interface options, USB or RS-232, but not both. 2. Place C101 and C102 physically close to U101. 3. For USB interface, place C109 and C110 physically close to U103. 4. For RS-232 interface, locate C103 - C107 physically close to U102. 5. This example uses hardware flow control!"
- title: 03 UART DMA RX Buffer -> FVR 01 Reference Bring Up
