File: 06 FVR/FVR 01 Reference Bring Up/FVR 01 Reference Bring Up.kicad_sch (KiCad schematic)
At the start: 24 parts, among them J101 ICSP, J102 USB_A, J103 DE9_Pins, U101 PIC18F47Q43-I/PT, U102 MAX232, U103 FT232RL

Commit message: FVR
Parts:
- added TP1: FVR Voltage, symbol Connector:TestPoint
Connections:
- net at U101.21 (RA2): now also TP1.1
- no-connect marks 47 -> 46
Changed lines of the file:
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@@
-	)
-	(no_connect
-		(at 60.96 62.23)
 	)
 	(no_connect
@@
 	(wire
 		(pts
+			(xy 57.15 46.99) (xy 57.15 62.23)
+		)
+		(stroke
+			(width 0)
+			(type default)
+		)
+	)
+	(wire
+		(pts
 			(xy 203.2 124.46) (xy 231.14 124.46)
 		)
@@
 		(pts
 			(xy 104.14 115.57) (xy 110.49 115.57)
+		)
+		(stroke
+			(width 0)
+			(type default)
+		)
+	)
+	(wire
+		(pts
+			(xy 57.15 62.23) (xy 60.96 62.23)
 		)
 		(stroke
@@
 					(unit 1)
 				)
+			)
+		)
+	)
+	(symbol
+		(lib_id "Connector:TestPoint")
+		(at 57.15 46.99 0)
+		(unit 1)
+		(body_style 1)
+		(exclude_from_sim no)
+		(in_bom yes)
+		(on_board yes)
+		(in_pos_files yes)
+		(dnp no)
+		(fields_autoplaced yes)
+		(property "Reference" "TP1"
+			(at 59.69 42.4179 0)
+			(show_name no)
+			(do_not_autoplace no)
+			(effects
+				(font
+					(size 1.27 1.27)
+				)
+				(justify left)
+			)
+		)
+		(property "Value" "FVR Voltage"
+			(at 59.69 44.9579 0)
+			(show_name no)
+			(do_not_autoplace no)
+			(effects
+				(font
+					(size 1.27 1.27)
+				)
+				(justify left)
+			)
+		)
+		(property "Footprint" ""
+			(at 62.23 46.99 0)
+			(hide yes)
+			(show_name no)
+			(do_not_autoplace no)
+			(effects
+				(font
+					(size 1.27 1.27)
+				)
+			)
+		)
+		(property "Datasheet" ""
+			(at 62.23 46.99 0)
+			(hide yes)
+			(show_name no)
+			(do_not_autoplace no)
+			(effects
+				(font
+					(size 1.27 1.27)
+				)
+			)
+		)
+		(property "Description" "test point"
+			(at 57.15 46.99 0)
+			(hide yes)
+			(show_name no)
+			(do_not_autoplace no)
+			(effects
+				(font
+					(size 1.27 1.27)
+				)
+			)
+		)
+		(pin "1"
+		)
+		(instances
+			(project "FVR 01 Reference Bring Up"
+				(path "/d3b5dd27-4845-413f-badb-7f64f7fb8d77"
+					(reference "TP1")
+					(unit 1)
+				)
