File: 07 ADCC DAC/ADCC 01 Window Comparator Hysteresis/ADCC 01 Window Comparator Hysteresis.kicad_sch (KiCad schematic)
At the start: 22 parts, among them J101 ICSP, J102 USB_A, J103 DB9_Pins, U101 PIC18F47Q43-I/PT, U102 MAX232, U103 FT232RL

Commit message: Added more examples
Co-authored-by: Copilot <copilot@github.com>
Parts:
- removed C103, C104, C106, C107, C108: 1, symbol Device:C_Polarized_Small_US
- removed J103: DB9_Pins, symbol Connector:DE9_Pins
- removed U102: MAX232, symbol Interface_UART:MAX232
- added D103: Window, symbol Device:LED_Small
- added R105: 270, symbol Device:R_US
- added RV1: 10K, symbol Device:R_Potentiometer_US
Connections:
- net +5V: now also D103.2 (A), RV1.1
- net GND: now also RV1.3
- net AD_IN: now reaches U101.19 (RA0)
- net AD_IN: now also RV1.2
- net CTS: no longer names the net of U101.11 (RB3)
- net CTS: no longer U103.3 (RTS)
- net RTS: no longer names the net of U101.10 (RB2)
- net RTS: now also R105.2; no longer U103.11 (CTS)
- new net: D103.1 (K), R105.1
Other:
- note added: "NOTE: A common mistake is to wire the controllers TX output to the TX pin of the FT232. The FT232 is labeled from the perspective of a remote device you want to connect to, so the FT232 TX pin should be connected to the controllers RX input, FT232 RX pin to the controllers TX output, etc. This is NOT the case when using an RS232 level shifter such as the MAX232, which is simply translating the si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"
- note added: "Notes: 1. Implement one or the other interface options, USB or RS-232, but not both. 2. Place C101 and C102 physically close to U101. 3. For USB interface, place C109 and C110 physically close to U103. 4. For RS-232 interface, locate C103 - C107 physically close to U102. 5. This example does not use hardware or software flow control!"
- note removed: "NOTE: A common mistake is to wire the controllers TX output to the TX pin of the FT232. The FT232 is labeled from the perspective of a remote device you want to connect to, so the FT232 TX pin should be connected to the controllers RX input, FT232 RX pin to the controllers TX output, etc. Cross connect RTS and CTS as well. This is NOT the case when using an RS232 level shifter such as the MAX232,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"
- note removed: "Notes: 1. Implement one or the other interface options, USB or RS-232, but not both. 2. Place C101 and C102 physically close to U101. 3. For USB interface, place C109 and C110 physically close to U103. 4. For RS-232 interface, locate C103 - C107 physically close to U102. 5. This example uses hardware flow control!"
- note removed: "RS-232 Interface"
- title: 03 UART DMA RX Buffer -> ADCC 01 Window Comparator Hysteresis
