File: 07 ADCC DAC/ADCC 01 Window Comparator Hysteresis/ADCC 01 Window Comparator Hysteresis.kicad_sch (KiCad schematic)
At the start: 18 parts, among them J101 ICSP, J102 USB_A, U101 PIC18F47Q43-I/PT, U103 FT232RL

Commit message: ADCC
Parts:
- added D104: HIGH, symbol Device:LED_Small
- added D105: WINDOW, symbol Device:LED_Small
- added R106, R107: 270, symbol Device:R_US
- D103: value Window -> LOW
Connections:
- net +5V: now also D104.2 (A), D105.2 (A)
- net at U101.11 (RB3): now also R106.2
- net at U101.14 (RB4): now also R107.2
- new net: D104.1 (K), R106.1
- new net: D105.1 (K), R107.1
- no-connect marks 40 -> 38
Other:
- note added: "This project uses the ADCC as a window comparator that verifies the input analog signal is between 2 and 3 volts DC. If it is below the window low threshold, the LOW LED is illuminated. If it is above the window upper threshold, the HIGH LED is illuminated. If it is within the window, the WINDOW LED is illuminated."
- note removed: "NOTE: A common mistake is to wire the controllers TX output to the TX pin of the FT232. The FT232 is labeled from the perspective of a remote device you want to connect to, so the FT232 TX pin should be connected to the controllers RX input, FT232 RX pin to the controllers TX output, etc. This is NOT the case when using an RS232 level shifter such as the MAX232, which is simply translating the si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"
- note removed: "Notes: 1. Implement one or the other interface options, USB or RS-232, but not both. 2. Place C101 and C102 physically close to U101. 3. For USB interface, place C109 and C110 physically close to U103. 4. For RS-232 interface, locate C103 - C107 physically close to U102. 5. This example does not use hardware or software flow control!"
- moved on the sheet: C101, C102, D103, R105, U101

Commit message: ADCC
Other:
- note added: "Note: The maximum source impedance recommended for the AD inputs is 10K. If the source impedance is higher than this, or if faster conversions are desired, this input should be buffered. Note, using a 10K pot gives us a max input source impedance of 5K since the impedance is seen from the input pin to either Vss or Vdd. The ADC acquisition time configuration MAY need to be adjusted if this value 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"
Changed lines of the file:
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@@
 		(company "Dewayne Hafenstein")
+	)
+	(text "Note: The maximum source impedance recommended for the AD inputs is \n10K.  If the source impedance is higher than this, or if faster \nconversions are desired, this input should be buffered.  Note, using\na 10K pot gives us a max input source impedance of 5K since the impedance\nis seen from the input pin to either Vss or Vdd.  The ADC acquisition \ntime configuration MAY need to be adjusted if this value is changed."
+		(exclude_from_sim no)
+		(at 147.574 41.148 0)
+		(effects
+			(font
+				(size 1.27 1.27)
+			)
+			(justify left)
+		)
 	)
 	(text "This project uses the ADCC as a window comparator that verifies the input analog \nsignal is between 2 and 3 volts DC.  If it is below the window low threshold, the LOW \nLED is illuminated.  If it is above the window upper threshold, the HIGH LED \nis illuminated.  If it is within the window, the WINDOW LED is illuminated."
