File: 01 UART/UART 02 DMA TX/UART 02 DMA TX.kicad_sch (KiCad schematic)
At the start: 15 parts, among them J101 ICSP, J102 USB_A, U101 PIC18F47Q43-I/PT, U103 FT232RL

Commit message: small edits
Other:
- title: 02 UART DMA TX Steam -> 02 UART DMA TX
