File: 01 UART/UART 02 DMA TX/UART 02 DMA TX.kicad_sch (KiCad schematic)
At the start: 15 parts, among them J101 ICSP, J102 USB_A, U101 PIC18F47Q43-I/PT, U103 FT232RL

Commit message: Updates
Parts:
- renumbered C105 to C103, C109 to C104, C110 to C105, R103 to R101, R101 to R102, R102 to R103, U103 to U102
Changed lines of the file:
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@@
 		(in_pos_files yes)
 		(dnp no)
-		(property "Reference" "#PWR0117"
+		(property "Reference" "#PWR0109"
 			(at 238.76 142.24 0)
 			(hide yes)
@@
 			(project "UART 02 DMA TX"
 				(path "/d3b5dd27-4845-413f-badb-7f64f7fb8d77"
-					(reference "#PWR0117")
+					(reference "#PWR0109")
 					(unit 1)
 				)
@@
 		(in_pos_files yes)
 		(dnp no)
-		(property "Reference" "#PWR0106"
+		(property "Reference" "#PWR0105"
 			(at 114.3 71.12 0)
 			(hide yes)
@@
 			(project "UART 02 DMA TX"
 				(path "/d3b5dd27-4845-413f-badb-7f64f7fb8d77"
-					(reference "#PWR0106")
+					(reference "#PWR0105")
 					(unit 1)
 				)
@@
 		(in_pos_files yes)
 		(dnp no)
-		(property "Reference" "#PWR0116"
+		(property "Reference" "#PWR0113"
 			(at 234.95 165.1 0)
 			(hide yes)
@@
 			(project "UART 02 DMA TX"
 				(path "/d3b5dd27-4845-413f-badb-7f64f7fb8d77"
-					(reference "#PWR0116")
+					(reference "#PWR0113")
 					(unit 1)
 				)
@@
 		(dnp no)
 		(fields_autoplaced yes)
-		(property "Reference" "#PWR0114"
+		(property "Reference" "#PWR0112"
 			(at 223.52 156.21 0)
 			(hide yes)
@@
 			(project "UART 02 DMA TX"
 				(path "/d3b5dd27-4845-413f-badb-7f64f7fb8d77"
-					(reference "#PWR0114")
+					(reference "#PWR0112")
 					(unit 1)
 				)
@@
 		(dnp no)
 		(fields_autoplaced yes)
-		(property "Reference" "#PWR0108"
+		(property "Reference" "#PWR0114"
 			(at 177.8 167.64 0)
 			(hide yes)
@@
 			(project "UART 02 DMA TX"
 				(path "/d3b5dd27-4845-413f-badb-7f64f7fb8d77"
-					(reference "#PWR0108")
+					(reference "#PWR0114")
 					(unit 1)
 				)
@@
 		(in_pos_files yes)
 		(dnp no)
-		(property "Reference" "#PWR0109"
+		(property "Reference" "#PWR0106"
 			(at 180.34 106.68 0)
 			(hide yes)
@@
 			(project "UART 02 DMA TX"
 				(path "/d3b5dd27-4845-413f-badb-7f64f7fb8d77"
-					(reference "#PWR0109")
+					(reference "#PWR0106")
 					(unit 1)
 				)
@@
 		(dnp no)
 		(fields_autoplaced yes)
-		(property "Reference" "#PWR0107"
+		(property "Reference" "#PWR0110"
 			(at 140.97 140.97 0)
 			(hide yes)
@@
 			(project "UART 02 DMA TX"
 				(path "/d3b5dd27-4845-413f-badb-7f64f7fb8d77"
-					(reference "#PWR0107")
+					(reference "#PWR0110")
 					(unit 1)
 				)
@@
 		(dnp no)
 		(fields_autoplaced yes)
-		(property "Reference" "R103"
+		(property "Reference" "R101"
 			(at 226.06 130.8099 0)
 			(show_name no)
@@
 			(project "UART 02 DMA TX"
 				(path "/d3b5dd27-4845-413f-badb-7f64f7fb8d77"
-					(reference "R103")
+					(reference "R101")
 					(unit 1)
 				)
@@
 		(in_pos_files yes)
 		(dnp no)
-		(property "Reference" "#PWR0105"
+		(property "Reference" "#PWR0104"
 			(at 114.3 55.88 0)
 			(hide yes)
@@
 			(project "UART 02 DMA TX"
 				(path "/d3b5dd27-4845-413f-badb-7f64f7fb8d77"
-					(reference "#PWR0105")
+					(reference "#PWR0104")
 					(unit 1)
 				)
@@
 		(in_pos_files yes)
 		(dnp no)
-		(property "Reference" "R101"
+		(property "Reference" "R102"
 			(at 148.082 135.636 90)
 			(show_name no)
@@
 			(project "UART 02 DMA TX"
 				(path "/d3b5dd27-4845-413f-badb-7f64f7fb8d77"
-					(reference "R101")
+					(reference "R102")
 					(unit 1)
 				)
@@
 		(in_pos_files yes)
 		(dnp no)
-		(property "Reference" "#PWR0115"
+		(property "Reference" "#PWR0111"
 			(at 234.95 149.86 0)
 			(hide yes)
@@
 			(project "UART 02 DMA TX"
 				(path "/d3b5dd27-4845-413f-badb-7f64f7fb8d77"
-					(reference "#PWR0115")
+					(reference "#PWR0111")
 					(unit 1)
 				)
@@
 		(dnp no)
 		(fields_autoplaced yes)
-		(property "Reference" "#PWR0104"
+		(property "Reference" "#PWR0108"
 			(at 106.68 134.62 0)
 			(hide yes)
@@
 			(project "UART 02 DMA TX"
 				(path "/d3b5dd27-4845-413f-badb-7f64f7fb8d77"
-					(reference "#PWR0104")
+					(reference "#PWR0108")
 					(unit 1)
 				)
@@
 		(in_pos_files yes)
 		(dnp no)
-		(property "Reference" "C110"
+		(property "Reference" "C105"
 			(at 243.332 148.336 0)
 			(show_name no)
@@
 			(project "UART 02 DMA TX"
 				(path "/d3b5dd27-4845-413f-badb-7f64f7fb8d77"
-					(reference "C110")
+					(reference "C105")
 					(unit 1)
 				)
@@
 		(in_pos_files yes)
 		(dnp no)
-		(property "Reference" "C109"
+		(property "Reference" "C104"
 			(at 235.458 148.844 0)
 			(show_name no)
@@
 			(project "UART 02 DMA TX"
 				(path "/d3b5dd27-4845-413f-badb-7f64f7fb8d77"
-					(reference "C109")
+					(reference "C104")
 					(unit 1)
 				)
@@
 		(in_pos_files yes)
 		(dnp no)
-		(property "Reference" "U103"
+		(property "Reference" "U102"
 			(at 178.1967 105.41 0)
 			(show_name no)
@@
 			(project "UART 02 DMA TX"
 				(path "/d3b5dd27-4845-413f-badb-7f64f7fb8d77"
-					(reference "U103")
+					(reference "U102")
 					(unit 1)
 				)
@@
 		(in_pos_files yes)
 		(dnp no)
-		(property "Reference" "R102"
+		(property "Reference" "R103"
 			(at 147.828 144.78 90)
 			(show_name no)
@@
 			(project "UART 02 DMA TX"
 				(path "/d3b5dd27-4845-413f-badb-7f64f7fb8d77"
-					(reference "R102")
+					(reference "R103")
 					(unit 1)
 				)
@@
 		(dnp no)
 		(fields_autoplaced yes)
-		(property "Reference" "#PWR0113"
+		(property "Reference" "#PWR0107"
 			(at 219.71 121.92 0)
 			(hide yes)
@@
 			(project "UART 02 DMA TX"
 				(path "/d3b5dd27-4845-413f-badb-7f64f7fb8d77"
-					(reference "#PWR0113")
+					(reference "#PWR0107")
 					(unit 1)
 				)
@@
 		(dnp no)
 		(fields_autoplaced yes)
-		(property "Reference" "C105"
+		(property "Reference" "C103"
 			(at 211.074 106.68 90)
 			(show_name no)
@@
 			(project "UART 02 DMA TX"
 				(path "/d3b5dd27-4845-413f-badb-7f64f7fb8d77"
-					(reference "C105")
-					(unit 1)
-				)
+					(reference "C103")
+					(unit 1)
+				)
