File: 01 UART/UART 03 DMA RX/UART 03 DMA RX.kicad_sch (KiCad schematic)
At the start: 22 parts, among them J101 ICSP, J102 USB_A, J103 DB9_Pins, U101 PIC18F47Q43-I/PT, U102 MAX232, U103 FT232RL

Commit message: small edits
Connections:
- net CTS renamed UART1_CTS
- net RTS renamed UART1_RTS
- net RxD renamed Receive_Data
- net TxD renamed Send_Data
Changed lines of the file:
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@@
 	(text "NOTE:  A common mistake is to wire the controllers TX output to the TX\npin of the FT232.  The  FT232 is labeled from the perspective of a remote\ndevice you want to connect to, so the FT232 TX pin should be connected to\nthe controllers RX input, FT232 RX pin to the controllers TX output, etc.\nCross connect RTS and CTS as well. \n\nThis is NOT the case when using an RS232 level shifter such as the \nMAX232, which is simply translating the signals to RS-232 levels. "
 		(exclude_from_sim no)
-		(at 63.246 187.96 0)
+		(at 30.734 177.038 0)
 		(effects
 			(font
@@
 	(wire
 		(pts
+			(xy 232.41 62.23) (xy 219.71 62.23)
+		)
+		(stroke
+			(width 0)
+			(type default)
+		)
+	)
+	(wire
+		(pts
 			(xy 201.93 46.99) (xy 209.55 46.99)
 		)
@@
 	(wire
 		(pts
-			(xy 242.57 147.32) (xy 234.95 147.32)
+			(xy 222.25 54.61) (xy 222.25 72.39)
 		)
 		(stroke
@@
 	(wire
 		(pts
-			(xy 212.09 62.23) (xy 212.09 59.69)
+			(xy 242.57 147.32) (xy 234.95 147.32)
 		)
 		(stroke
@@
 	(wire
 		(pts
+			(xy 201.93 59.69) (xy 219.71 59.69)
+		)
+		(stroke
+			(width 0)
+			(type default)
+		)
+	)
+	(wire
+		(pts
 			(xy 121.92 54.61) (xy 121.92 53.34)
 		)
@@
 	(wire
 		(pts
+			(xy 219.71 59.69) (xy 219.71 62.23)
+		)
+		(stroke
+			(width 0)
+			(type default)
+		)
+	)
+	(wire
+		(pts
 			(xy 139.7 119.38) (xy 162.56 119.38)
 		)
@@
 	(wire
 		(pts
-			(xy 201.93 59.69) (xy 212.09 59.69)
-		)
-		(stroke
-			(width 0)
-			(type default)
-		)
-	)
-	(wire
-		(pts
 			(xy 241.3 134.62) (xy 238.76 134.62)
 		)
@@
 	(wire
 		(pts
-			(xy 222.25 72.39) (xy 222.25 54.61)
-		)
-		(stroke
-			(width 0)
-			(type default)
-		)
-	)
-	(wire
-		(pts
 			(xy 33.02 85.09) (xy 60.96 85.09)
 		)
@@
 	(wire
 		(pts
-			(xy 232.41 62.23) (xy 212.09 62.23)
-		)
-		(stroke
-			(width 0)
-			(type default)
-		)
-	)
-	(wire
-		(pts
 			(xy 222.25 34.29) (xy 222.25 24.13)
 		)
@@
 		)
 	)
-	(label "RTS"
+	(label "UART1_RTS"
 		(at 33.02 87.63 0)
 		(effects
@@
 		)
 	)
-	(label "RTS"
+	(label "UART1_RTS"
 		(at 140.97 74.93 0)
 		(effects
@@
 		)
 	)
-	(label "TxD"
+	(label "Send_Data"
 		(at 203.2 59.69 0)
 		(effects
@@
 		)
 	)
-	(label "CTS"
+	(label "UART1_CTS"
 		(at 33.02 90.17 0)
 		(effects
@@
 		)
 	)
-	(label "RxD"
+	(label "Receive_Data"
 		(at 203.2 69.85 0)
 		(effects
@@
 		)
 	)
-	(label "CTS"
+	(label "UART1_CTS"
 		(at 140.97 64.77 0)
 		(effects
@@
 		)
 	)
-	(label "RTS"
+	(label "UART1_RTS"
 		(at 139.7 121.92 0)
 		(effects
@@
 		)
 	)
-	(label "CTS"
+	(label "UART1_CTS"
 		(at 139.7 119.38 0)
 		(effects
@@
 		)
 		(instances
-			(project "UART 03 DMA RX Buffer"
+			(project "UART 03 DMA RX"
 				(path "/d3b5dd27-4845-413f-badb-7f64f7fb8d77"
 					(reference "D102")
@@
 		)
 		(instances
-			(project "UART 03 DMA RX Buffer"
+			(project "UART 03 DMA RX"
 				(path "/d3b5dd27-4845-413f-badb-7f64f7fb8d77"
 					(reference "#PWR0117")
@@
 		)
 		(instances
-			(project "UART 03 DMA RX Buffer"
+			(project "UART 03 DMA RX"
 				(path "/d3b5dd27-4845-413f-badb-7f64f7fb8d77"
 					(reference "#PWR0106")
@@
 		)
 		(instances
-			(project "UART 03 DMA RX Buffer"
+			(project "UART 03 DMA RX"
 				(path "/d3b5dd27-4845-413f-badb-7f64f7fb8d77"
 					(reference "#PWR0112")
@@
 		)
 		(instances
-			(project "UART 03 DMA RX Buffer"
+			(project "UART 03 DMA RX"
 				(path "/d3b5dd27-4845-413f-badb-7f64f7fb8d77"
 					(reference "C102")
@@
 		)
 		(instances
-			(project "UART 03 DMA RX Buffer"
+			(project "UART 03 DMA RX"
 				(path "/d3b5dd27-4845-413f-badb-7f64f7fb8d77"
 					(reference "#PWR0101")
@@
 		)
 		(instances
-			(project "UART 03 DMA RX Buffer"
+			(project "UART 03 DMA RX"
 				(path "/d3b5dd27-4845-413f-badb-7f64f7fb8d77"
 					(reference "#PWR0116")
@@
 		)
 		(instances
-			(project "UART 03 DMA RX Buffer"
+			(project "UART 03 DMA RX"
 				(path "/d3b5dd27-4845-413f-badb-7f64f7fb8d77"
 					(reference "#PWR0114")
@@
 		)
 		(instances
-			(project "UART 03 DMA RX Buffer"
+			(project "UART 03 DMA RX"
 				(path "/d3b5dd27-4845-413f-badb-7f64f7fb8d77"
 					(reference "J101")
@@
 		)
 		(instances
-			(project "UART 03 DMA RX Buffer"
+			(project "UART 03 DMA RX"
 				(path "/d3b5dd27-4845-413f-badb-7f64f7fb8d77"
 					(reference "#PWR0102")
@@
 		)
 		(instances
-			(project "UART 03 DMA RX Buffer"
+			(project "UART 03 DMA RX"
 				(path "/d3b5dd27-4845-413f-badb-7f64f7fb8d77"
 					(reference "#PWR0103")
@@
 		)
 		(instances
-			(project "UART 03 DMA RX Buffer"
+			(project "UART 03 DMA RX"
 				(path "/d3b5dd27-4845-413f-badb-7f64f7fb8d77"
 					(reference "C103")
@@
 		)
 		(instances
-			(project "UART 03 DMA RX Buffer"
+			(project "UART 03 DMA RX"
 				(path "/d3b5dd27-4845-413f-badb-7f64f7fb8d77"
 					(reference "J103")
@@
 		)
 		(instances
-			(project "UART 03 DMA RX Buffer"
+			(project "UART 03 DMA RX"
 				(path "/d3b5dd27-4845-413f-badb-7f64f7fb8d77"
 					(reference "#PWR0108")
@@
 		)
 		(instances
-			(project "UART 03 DMA RX Buffer"
+			(project "UART 03 DMA RX"
 				(path "/d3b5dd27-4845-413f-badb-7f64f7fb8d77"
 					(reference "#PWR0109")
@@
 		)
 		(instances
-			(project "UART 03 DMA RX Buffer"
+			(project "UART 03 DMA RX"
 				(path "/d3b5dd27-4845-413f-badb-7f64f7fb8d77"
 					(reference "#PWR0107")
@@
 		)
 		(instances
-			(project "UART 03 DMA RX Buffer"
+			(project "UART 03 DMA RX"
 				(path "/d3b5dd27-4845-413f-badb-7f64f7fb8d77"
 					(reference "R103")
@@
 		)
 		(instances
-			(project "UART 03 DMA RX Buffer"
+			(project "UART 03 DMA RX"
 				(path "/d3b5dd27-4845-413f-badb-7f64f7fb8d77"
 					(reference "D101")
@@
 		)
 		(instances
-			(project "UART 03 DMA RX Buffer"
+			(project "UART 03 DMA RX"
 				(path "/d3b5dd27-4845-413f-badb-7f64f7fb8d77"
 					(reference "C101")
@@
 		)
 		(instances
-			(project "UART 03 DMA RX Buffer"
+			(project "UART 03 DMA RX"
 				(path "/d3b5dd27-4845-413f-badb-7f64f7fb8d77"
 					(reference "C108")
@@
 		)
 		(instances
-			(project "UART 03 DMA RX Buffer"
+			(project "UART 03 DMA RX"
 				(path "/d3b5dd27-4845-413f-badb-7f64f7fb8d77"
 					(reference "C107")
@@
 		)
 		(instances
-			(project "UART 03 DMA RX Buffer"
+			(project "UART 03 DMA RX"
 				(path "/d3b5dd27-4845-413f-badb-7f64f7fb8d77"
 					(reference "#PWR0110")
@@
 		)
 		(instances
-			(project "UART 03 DMA RX Buffer"
+			(project "UART 03 DMA RX"
 				(path "/d3b5dd27-4845-413f-badb-7f64f7fb8d77"
 					(reference "#PWR0105")
@@
 		)
 		(instances
-			(project "UART 03 DMA RX Buffer"
+			(project "UART 03 DMA RX"
 				(path "/d3b5dd27-4845-413f-badb-7f64f7fb8d77"
 					(reference "R101")
@@
 		)
 		(instances
-			(project "UART 03 DMA RX Buffer"
+			(project "UART 03 DMA RX"
 				(path "/d3b5dd27-4845-413f-badb-7f64f7fb8d77"
 					(reference "R104")
@@
 		)
 		(instances
-			(project "UART 03 DMA RX Buffer"
+			(project "UART 03 DMA RX"
 				(path "/d3b5dd27-4845-413f-badb-7f64f7fb8d77"
 					(reference "#PWR0115")
@@
 		)
 		(instances
-			(project "UART 03 DMA RX Buffer"
+			(project "UART 03 DMA RX"
 				(path "/d3b5dd27-4845-413f-badb-7f64f7fb8d77"
 					(reference "#PWR0111")
@@
 		)
 		(instances
-			(project "UART 03 DMA RX Buffer"
+			(project "UART 03 DMA RX"
 				(path "/d3b5dd27-4845-413f-badb-7f64f7fb8d77"
 					(reference "J102")
@@
 		)
 		(instances
-			(project "UART 03 DMA RX Buffer"
+			(project "UART 03 DMA RX"
 				(path "/d3b5dd27-4845-413f-badb-7f64f7fb8d77"
 					(reference "U102")
@@
 		)
 		(instances
-			(project "UART 03 DMA RX Buffer"
+			(project "UART 03 DMA RX"
 				(path "/d3b5dd27-4845-413f-badb-7f64f7fb8d77"
 					(reference "C104")
@@
 		)
 		(instances
-			(project "UART 03 DMA RX Buffer"
+			(project "UART 03 DMA RX"
 				(path "/d3b5dd27-4845-413f-badb-7f64f7fb8d77"
 					(reference "C106")
@@
 		)
 		(instances
-			(project "UART 03 DMA RX Buffer"
+			(project "UART 03 DMA RX"
 				(path "/d3b5dd27-4845-413f-badb-7f64f7fb8d77"
 					(reference "U101")
@@
 		)
 		(instances
-			(project "UART 03 DMA RX Buffer"
+			(project "UART 03 DMA RX"
 				(path "/d3b5dd27-4845-413f-badb-7f64f7fb8d77"
 					(reference "#PWR0104")
@@
 		)
 		(instances
-			(project "UART 03 DMA RX Buffer"
+			(project "UART 03 DMA RX"
 				(path "/d3b5dd27-4845-413f-badb-7f64f7fb8d77"
 					(reference "C110")
@@
 		)
 		(instances
-			(project "UART 03 DMA RX Buffer"
+			(project "UART 03 DMA RX"
 				(path "/d3b5dd27-4845-413f-badb-7f64f7fb8d77"
 					(reference "C109")
@@
 		)
 		(instances
-			(project "UART 03 DMA RX Buffer"
+			(project "UART 03 DMA RX"
 				(path "/d3b5dd27-4845-413f-badb-7f64f7fb8d77"
 					(reference "U103")
@@
 		)
 		(instances
-			(project "UART 03 DMA RX Buffer"
+			(project "UART 03 DMA RX"
 				(path "/d3b5dd27-4845-413f-badb-7f64f7fb8d77"
 					(reference "R102")
@@
 		)
 		(instances
-			(project "UART 03 DMA RX Buffer"
+			(project "UART 03 DMA RX"
 				(path "/d3b5dd27-4845-413f-badb-7f64f7fb8d77"
 					(reference "#PWR0113")
@@
 		)
 		(instances
-			(project "UART 03 DMA RX Buffer"
+			(project "UART 03 DMA RX"
 				(path "/d3b5dd27-4845-413f-badb-7f64f7fb8d77"
 					(reference "C105")
