File: 03 I2C/I2C 03 Module Slave/I2C 01 Module Slave.kicad_sch (KiCad schematic)
At the start: 22 parts, among them J101 ICSP Master, J102 USB_A, J103 ICSP Slave, SW101 SW_DIP_x08, U101 PIC18F47Q43-I/PT, U102 PIC18F47Q43-I/PT, U103 FT232RL

Commit message: i2c
Parts:
- removed U101: PIC18F47Q43-I/PT, Package_QFP:TQFP-44_10x10mm_P0.8mm, symbol DH_MCU_Microchip:PIC18F47Q43-I/PT
- added D103: TX, symbol Device:LED_Small
- added D104: RX, symbol Device:LED_Small
- added R105, R106: 330, symbol Device:R_US
- added U1: PIC18F27Q43, symbol DH_MCU_Microchip:PIC18F27Q43
- R101, R102: value 270 -> 330
Connections:
- net +5V: now also R105.1, R106.1, U1.20 (Vdd)
- net GND: now also U1.19 (Vss), U1.8 (Vss)
- net IOC: now also U1.23 (RB2)
- net SCK: now also U1.14 (RC3)
- net SDA: now also U1.15 (RC4)
- net UART1_RX: now also U1.22 (RB1)
- net UART1_TX: now also U1.21 (RB0)
- net at J101.4 (Pin_4): now also U1.28 (RB7/ICSPDAT)
- net at J101.5 (Pin_5): now also U1.27 (RB6/ICSPCLK)
- net at U102.1 (RC7): now also D104.1 (K)
- net at U102.44 (RC6): now also D103.1 (K)
- net ~{RESET}: no longer names the net of J101.1 (Pin_1)
- net ~{RESET}: now also U1.1 (~{MCLR})
- new net: D103.2 (A), R105.2
- new net: D104.2 (A), R106.2
- no-connect marks 48 -> 37
Other:
- note added: "In this example slave device, RC0..2 are used as the address selection pins. The device has a base address of x'10'"
- moved on the sheet: C101, C102, J103
