File: 03 I2C/I2C 04 Module Master DMA/I2C 01 Module Master.kicad_sch (KiCad schematic)
At the start: 19 parts, among them J101 ICSP, J102 USB_A, SW101 SW_DIP_x08, U101 PIC18F47Q43-I/PT, U102 MCP23017_SO, U103 FT232RL

Commit message: i2c
Parts:
- removed U101: PIC18F47Q43-I/PT, Package_QFP:TQFP-44_10x10mm_P0.8mm, symbol DH_MCU_Microchip:PIC18F47Q43-I/PT
- removed U102: MCP23017_SO, Package_SO:SOIC-28W_7.5x17.9mm_P1.27mm, symbol DH_Interface:MCP23017_SO
- added C103: 4.7, symbol Device:C_Polarized_Small_US
- added C104: 100n, symbol Device:C_US
- added D103: TX, symbol Device:LED_Small
- added D104: RX, symbol Device:LED_Small
- added J103: ICSP Slave, symbol Connector_Generic:Conn_01x05
- added R105, R106: 330, symbol Device:R_US
- added U1: PIC18F27Q43, symbol DH_MCU_Microchip:PIC18F27Q43
- added U102: PIC18F47Q43-I/PT, Package_QFP:TQFP-44_10x10mm_P0.8mm, symbol DH_MCU_Microchip:PIC18F47Q43-I/PT
- J101: value ICSP -> ICSP Master
- R101, R102: value 270 -> 330
Connections:
- net +5V: now also C103.1, C104.1, J103.2 (Pin_2), R105.1, R106.1, U1.20 (Vdd), U102.28 (Vdd), U102.7 (Vdd)
- net GND: now also U103.18 (GND), C103.2, C104.2, J103.3 (Pin_3), U1.19 (Vss), U1.8 (Vss), U102.29 (Vss), U102.32 (RC0), U102.35 (RC1), U102.36 (RC2), U102.6 (Vss)
- net IOC: now also U1.23 (RB2), U102.8 (RB0)
- net SCK: now also U1.14 (RC3), U102.37 (RC3)
- net SDA: now also U1.15 (RC4), U102.42 (RC4)
- net UART1_RX: now also U1.22 (RB1)
- net UART1_TX: now also U1.21 (RB0)
- net at J101.4 (Pin_4): now also U1.28 (RB7/ICSPDAT)
- net at J101.5 (Pin_5): now also U1.27 (RB6/ICSPCLK)
- net at RN101.1 (R1.1): now also U102.38 (RD0)
- net at RN101.2 (R2.1): now also U102.39 (RD1)
- net at RN101.3 (R3.1): now also U102.40 (RD2)
- net at RN101.4 (R4.1): now also U102.41 (RD3)
- net at RN101.5 (R5.1): now also U102.2 (RD4)
- net at RN101.6 (R6.1): now also U102.3 (RD5)
- net at RN101.7 (R7.1): now also U102.4 (RD6)
- net at RN101.8 (R8.1): now also U102.5 (RD7)
- net at SW101.1: now also U102.19 (RA0)
- net at SW101.2: now also U102.20 (RA1)
- net at SW101.3: now also U102.21 (RA2)
- net at SW101.4: now also U102.22 (RA3)
- net at SW101.5: now also U102.23 (RA4)
- net at SW101.6: now also U102.24 (RA5)
- net at SW101.7: now also U102.31 (RA6)
- net at SW101.8: now also U102.30 (RA7)
- net ~{RESET}: no longer names the net of J101.1 (Pin_1)
- net ~{RESET}: now also U1.1 (~{MCLR})
- new net: D104.2 (A), R106.2
- new net: J103.1 (Pin_1), U102.18 (~{MCLR}/Vpp/RE3)
- new net: J103.4 (Pin_4), U102.17 (RB7/ICSPDAT)
- new net: J103.5 (Pin_5), U102.16 (RB6/ICSPCLK)
- new net: D103.2 (A), R105.2
- new net: D104.1 (K), U102.1 (RC7)
- new net: D103.1 (K), U102.44 (RC6)
- no-connect marks 42 -> 37
Other:
- note added: "In this example slave device, RC0..2 are used as the address selection pins. The device has a base address of x'10'."
- note added: "This example circuit uses another Q43 PIC as a slave device. The address of the slave is determined using RC0..2 inputs. Port A is the input switches, and port D is the output LED display. The slave generates an interrupt on change on port RB0 pin if any of the inputs change value. A smaller PIC device can be used as well depending on the inputs that need to be scanned or monitored as well as out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"
- note removed: "I had 10 LED bar displays and used the first 8. Discrete LEDs could also be used. I also used a Bourns 4116R-1-331 (330 ohm) resistor pack DIP. Individual resistors can also be used. A DIP switch is shown, but individual jumpers to ground could be used instead."
- note removed: "Note, the MCP23017 drives LEDs better by pulling the LED to ground. Therefore, signals are inverted in order to "turn on" an LED."
- note removed: "This example circuit uses an I/O expander (MCP2317) connected via I2C interface with interrupt on change enabled. It could also be polled periodically for changes."
- title: Module Master DMA -> Module Master
- moved on the sheet: BAR101, C101, C102, C105, C109, C110, D101, D102, J101, J102, R101, R102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
