File: 03 I2C/I2C 05 Module Slave DMA/I2C 01 Module Slave DMA.kicad_sch (KiCad schematic)
At the start: 22 parts, among them J101 ICSP Master, J102 USB_A, J103 ICSP Slave, SW101 SW_DIP_x08, U101 PIC18F47Q43-I/PT, U102 PIC18F47Q43-I/PT, U103 FT232RL

Commit message: i2c
Connections:
- net ~{RESET}: no longer names the net of J101.1 (Pin_1), U101.18 (~{MCLR}/Vpp/RE3)
Other:
- moved on the sheet: C109, C110, J102, R103, R104
