File: 04 SPI/SPI 01 Host/SPI 01 Host.kicad_sch (KiCad schematic)
At the start: 26 parts, among them J101 ICSP Master, J102 USB_A, J103 ICSP Slave, SW101 SW_DIP_x08, U1 PIC18F27Q43, U102 PIC18F47Q43-I/PT, U103 FT232RL

Commit message: SPI 01
Parts:
- removed C103: 4.7, symbol Device:C_Polarized_Small_US
- removed C104: 100n, symbol Device:C_US
- removed D103: TX, symbol Device:LED_Small
- removed D104: RX, symbol Device:LED_Small
- removed J103: ICSP Slave, symbol Connector_Generic:Conn_01x05
- removed R105, R106: 330, symbol Device:R_US
- removed U1: PIC18F27Q43, symbol DH_MCU_Microchip:PIC18F27Q43
- removed U102: PIC18F47Q43-I/PT, Package_QFP:TQFP-44_10x10mm_P0.8mm, symbol DH_MCU_Microchip:PIC18F47Q43-I/PT
- added U1: MCP23S17_SO, Package_SO:SOIC-28W_7.5x17.9mm_P1.27mm, symbol DH-:MCP23S17_SO
- added U101: PIC18F47Q43-I/PT, Package_QFP:TQFP-44_10x10mm_P0.8mm, symbol DH_MCU_Microchip:PIC18F47Q43-I/PT
- added U2: 74LS138, symbol 74xx:74LS138
- J101: value ICSP Master -> ICSP
- R101, R102: value 330 -> 270
Connections:
- net +5V: now also U1.18 (~{RESET}), U1.9 (VDD), U101.28 (Vdd), U101.7 (Vdd), U2.16 (VCC)
- net GND: now also U1.10 (VSS), U1.15 (A0), U1.16 (A1), U1.17 (A2), U101.29 (Vss), U101.6 (Vss), U2.4 (E1), U2.5 (E2), U2.8 (GND); no longer U103.18 (GND)
- net IOC: now also U1.20 (INTA), U101.10 (RB2)
- net UART1_RX: now also U101.9 (RB1)
- net UART1_TX: now also U101.8 (RB0)
- net at J101.1 (Pin_1): now also U101.18 (~{MCLR}/Vpp/RE3)
- net at J101.4 (Pin_4): now also U101.17 (RB7/ICSPDAT)
- net at J101.5 (Pin_5): now also U101.16 (RB6/ICSPCLK)
- net at SW101.1: now also U1.21 (GPA0)
- net at RN101.5 (R5.1): now also U1.5 (GPB4)
- net at SW101.2: now also U1.22 (GPA1)
- net at SW101.3: now also U1.23 (GPA2)
- net at SW101.4: now also U1.24 (GPA3)
- net at SW101.5: now also U1.25 (GPA4)
- net at SW101.6: now also U1.26 (GPA5)
- net at RN101.6 (R6.1): now also U1.6 (GPB5)
- net at SW101.8: now also U1.28 (GPA7)
- net at SW101.7: now also U1.27 (GPA6)
- net at RN101.1 (R1.1): now also U1.1 (GPB0)
- net at RN101.2 (R2.1): now also U1.2 (GPB1)
- net at RN101.7 (R7.1): now also U1.7 (GPB6)
- net at RN101.3 (R3.1): now also U1.3 (GPB2)
- net at RN101.4 (R4.1): now also U1.4 (GPB3)
- net at RN101.8 (R8.1): now also U1.8 (GPB7)
- new net: U1.11 (~{CS}), U2.15 (O0)
- new net A0: U101.32 (RC0), U2.1 (A0)
- new net A1: U101.35 (RC1), U2.2 (A1)
- new net A2: U101.36 (RC2), U2.3 (A2)
- new net SCLK: U1.12 (SCK), U101.37 (RC3)
- new net SDI: U1.14 (SO), U101.42 (RC4)
- new net SDO: U1.13 (SI), U101.43 (RC5)
- new net SS: U101.44 (RC6), U2.6 (E3)
- no-connect marks 37 -> 42
Other:
- note added: "0x00 0x01 0x02 0x03 0x04 0x05 0x06 0x07"
- note added: "Device 0X00"
- note added: "I had 10 LED bar displays and used the first 8. Discrete LEDs could also be used. I also used a Bourns 4116R-1-331 (330 ohm) resistor pack DIP. Individual resistors can also be used. A DIP switch is shown, but individual jumpers to ground could be used instead."
- note added: "Note, the MCP23S17 drives LEDs better by pulling the LED to ground. Therefore, signals are inverted in order to "turn on" an LED."
- note added: "This example circuit uses an I/O expander (MCP23S17) connected via SPI interface with interrupt on change enabled. It could also be polled periodically for changes. Note that SPI peripherals generally are selected using a "chip select" input. They are not usually addressed like the I2C versions (the MCP23S17 does offer this option as well), which requires the use of separate select lines for each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"
- note removed: "In this example slave device, RC0..2 are used as the address selection pins. The device has a base address of x'10'."
- note removed: "This example circuit uses another Q43 PIC as a slave device. The address of the slave is determined using RC0..2 inputs. Port A is the input switches, and port D is the output LED display. The slave generates an interrupt on change on port RB0 pin if any of the inputs change value. A smaller PIC device can be used as well depending on the inputs that need to be scanned or monitored as well as out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"
- title: Module Master -> SPI Host
- moved on the sheet: BAR101, C101, C102, C105, C109, C110, D101, D102, J101, J102, R101, R102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

Commit message: spi
Connections:
- net +5V: now also U2.6 (E3); no longer U1.18 (~{RESET})
- net GND: no longer U2.4 (E1)
- net ~{RESET}: now reaches U101.1 (RC7)
- net ~{RESET}: now also U1.18 (~{RESET})
- net SS renamed ~{SS}
- net ~{SS}: now also U2.4 (E1); no longer U2.6 (E3)
- no-connect marks 42 -> 41
Other:
- moved on the sheet: U2
