File: 07 ADCC DAC/DAC 01 Reference Ladder/DAC 01 Reference Ladder.kicad_sch (KiCad schematic)
At the start: 15 parts, among them J101 ICSP, J102 USB_A, U101 PIC18F47Q43-I/PT, U103 FT232RL

Commit message: updated schematic
Parts:
- added TP1: DAC_OUT, symbol Connector:TestPoint
Connections:
- net at U101.19 (RA0): no longer U101.20 (RA1)
- new net: TP1.1, U101.20 (RA1)
- no-connect marks 40 -> 41
Other:
- note added: "DAC output (RA1)"
- note removed: "DAC output (RA1) is looped back to ADCC input (RA0)"
- note removed: "NOTE: A common mistake is to wire the controllers TX output to the TX pin of the FT232. The FT232 is labeled from the perspective of a remote device you want to connect to, so the FT232 TX pin should be connected to the controllers RX input, FT232 RX pin to the controllers TX output, etc. This is NOT the case when using an RS232 level shifter such as the MAX232, which is simply translating the si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"
- note removed: "Notes: 1. Implement one or the other interface options, USB or RS-232, but not both. 2. Place C101 and C102 physically close to U101. 3. For USB interface, place C109 and C110 physically close to U103. 4. For RS-232 interface, locate C103 - C107 physically close to U102. 5. This example does not use hardware or software flow control!"
Changed lines of the file:
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@@
 		(company "Dewayne Hafenstein")
 	)
-	(text "DAC output (RA1) is looped\nback to ADCC input (RA0)"
+	(text "DAC output (RA1)"
 		(exclude_from_sim no)
-		(at 20.32 58.166 0)
-		(effects
-			(font
-				(size 1.27 1.27)
-			)
-			(justify left)
-		)
-	)
-	(text "NOTE:  A common mistake is to wire the controllers TX output to the TX\npin of the FT232.  The  FT232 is labeled from the perspective of a remote\ndevice you want to connect to, so the FT232 TX pin should be connected to\nthe controllers RX input, FT232 RX pin to the controllers TX output, etc. \n\nThis is NOT the case when using an RS232 level shifter such as the \nMAX232, which is simply translating the signals to RS-232 levels. "
-		(exclude_from_sim no)
-		(at 63.246 187.96 0)
-		(effects
-			(font
-				(size 1.27 1.27)
-			)
-			(justify left)
-		)
-	)
-	(text "Notes:\n1. Implement one or the other interface options, USB or RS-232,\n   but not both.\n2. Place C101 and C102 physically close to U101.\n3. For USB interface, place C109 and C110 physically close to U103.\n4. For RS-232 interface, locate C103 - C107 physically close to U102.\n5. This example does not use hardware or software flow control!"
-		(exclude_from_sim no)
-		(at 30.734 158.242 0)
+		(at 55.118 39.624 0)
 		(effects
 			(font
@@
 	)
 	(no_connect
+		(at 60.96 57.15)
+	)
+	(no_connect
 		(at 104.14 110.49)
 	)
@@
 		)
 	)
-	(bus
-		(pts
-			(xy 137.16 40.64) (xy 137.16 111.76)
-		)
-		(stroke
-			(width 0)
-			(type default)
-		)
-	)
 	(wire
 		(pts
@@
 	(wire
 		(pts
-			(xy 55.88 57.15) (xy 55.88 59.69)
-		)
-		(stroke
-			(width 0)
-			(type default)
-		)
-	)
-	(wire
-		(pts
 			(xy 104.14 57.15) (xy 106.68 57.15)
 		)
@@
 	(wire
 		(pts
-			(xy 60.96 57.15) (xy 55.88 57.15)
-		)
-		(stroke
-			(width 0)
-			(type default)
-		)
-	)
-	(wire
-		(pts
 			(xy 177.8 157.48) (xy 177.8 160.02)
 		)
@@
 		)
 	)
+	(bus
+		(pts
+			(xy 30.48 55.88) (xy 30.48 80.01)
+		)
+		(stroke
+			(width 0)
+			(type default)
+		)
+	)
 	(wire
 		(pts
@@
 		)
 	)
+	(bus
+		(pts
+			(xy 137.16 95.25) (xy 137.16 111.76)
+		)
+		(stroke
+			(width 0)
+			(type default)
+		)
+	)
 	(wire
 		(pts
@@
 	(wire
 		(pts
+			(xy 55.88 46.99) (xy 55.88 59.69)
+		)
+		(stroke
+			(width 0)
+			(type default)
+		)
+	)
+	(wire
+		(pts
 			(xy 106.68 54.61) (xy 106.68 52.07)
 		)
@@
 					(unit 1)
 				)
+			)
+		)
+	)
+	(symbol
+		(lib_id "Connector:TestPoint")
+		(at 55.88 46.99 0)
+		(unit 1)
+		(body_style 1)
+		(exclude_from_sim no)
+		(in_bom yes)
+		(on_board yes)
+		(in_pos_files yes)
+		(dnp no)
+		(fields_autoplaced yes)
+		(property "Reference" "TP1"
+			(at 58.42 42.4179 0)
+			(show_name no)
+			(do_not_autoplace no)
+			(effects
+				(font
+					(size 1.27 1.27)
+				)
+				(justify left)
+			)
+		)
+		(property "Value" "DAC_OUT"
+			(at 58.42 44.9579 0)
+			(show_name no)
+			(do_not_autoplace no)
+			(effects
+				(font
+					(size 1.27 1.27)
+				)
+				(justify left)
+			)
+		)
+		(property "Footprint" ""
+			(at 60.96 46.99 0)
+			(hide yes)
+			(show_name no)
+			(do_not_autoplace no)
+			(effects
+				(font
+					(size 1.27 1.27)
+				)
+			)
+		)
+		(property "Datasheet" ""
+			(at 60.96 46.99 0)
+			(hide yes)
+			(show_name no)
+			(do_not_autoplace no)
+			(effects
+				(font
+					(size 1.27 1.27)
+				)
+			)
+		)
+		(property "Description" "test point"
+			(at 55.88 46.99 0)
+			(hide yes)
+			(show_name no)
+			(do_not_autoplace no)
+			(effects
+				(font
+					(size 1.27 1.27)
+				)
+			)
+		)
+		(pin "1"
+		)
+		(instances
+			(project "DAC 01 Reference Ladder"
+				(path "/d3b5dd27-4845-413f-badb-7f64f7fb8d77"
+					(reference "TP1")
+					(unit 1)
+				)
