File: 08 Temp Indicator/Temp 02 Thermistor Linearization/Temp 02 Thermistor Linearization.kicad_sch (KiCad schematic)
At the start: 16 parts, among them J101 ICSP, J102 USB_A, U101 PIC18F47Q43-I/PT, U103 FT232RL

Commit message: temp
Parts:
- removed RV1: 10K, symbol Device:R_Potentiometer_US
- added R105: 4.42K, symbol Device:R_US
- added TH1: NTCDS3HG103HC3NB, symbol Device:Thermistor_US
Connections:
- net +5V: now also TH1.1
- net GND: now also R105.2
- net at U101.20 (RA1): no longer U101.21 (RA2)
- net SERVO_IN: no longer names the net of U101.19 (RA0)
- net SERVO_IN: now also R105.1, TH1.2
- no-connect marks 39 -> 41
Other:
- note added: "Note: There are several more ways to linearize a thermistor that are not shown. One approach (not shown) is to use a resistor in parallel with the thermistor that corrects its resistance at the center of the range your interested in. As you get further away from this central correction, the error will increase. This approach is convenient and easy, but reduces the dynamic range of the thermistor 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"
- note added: "The value of R105 is chosen to produce a voltage at the junction of less than 4.096V when the thermistor is at it's lowest resistance. For the values shown, using TDK NTCDS3HG103HC3NB, the range of voltages from 0C to 100C are approx 0.69V to 4.08V. Adjust the resistor for the thermistor you are using to produce a voltage less than 4.096V at full scale."
- note added: "Use a thermistor that reads about 10K at room temperature and has a negative temperature coefficient. This allows the sensed voltage to increase as the temperature increases (the NTC thermistor decreases in value). Calibrate the sensor at several temperatures if possible, such as freezing (0C or 32F), room temperature (25C or 77F), and boiling water (100C or 212F). This 3 point calibration should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"
- note removed: "NOTE: A common mistake is to wire the controllers TX output to the TX pin of the FT232. The FT232 is labeled from the perspective of a remote device you want to connect to, so the FT232 TX pin should be connected to the controllers RX input, FT232 RX pin to the controllers TX output, etc. This is NOT the case when using an RS232 level shifter such as the MAX232, which is simply translating the si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"
- note removed: "Notes: 1. Implement one or the other interface options, USB or RS-232, but not both. 2. Place C101 and C102 physically close to U101. 3. For USB interface, place C109 and C110 physically close to U103. 4. For RS-232 interface, locate C103 - C107 physically close to U102. 5. This example does not use hardware or software flow control!"
- title: DAC 02 Software Servo Threshold -> Temp 02 Thermistor Linearization
