File: 03 I2C/I2C 02 Module Host/I2C 01 Module Master.kicad_sch (KiCad schematic)
At the start: 19 parts, among them J101 ICSP, J102 USB_A, SW101 SW_DIP_x08, U101 PIC18F47Q43-I/PT, U102 MCP23017_SO, U103 FT232RL

Commit message: i2c
Connections:
- net ~{RESET}: now also U101.11 (RB3); no longer J101.1 (Pin_1), U101.18 (~{MCLR}/Vpp/RE3)
- new net: J101.1 (Pin_1), U101.18 (~{MCLR}/Vpp/RE3)
- no-connect marks 42 -> 41
