File: 03 I2C/I2C 02 Module Host/I2C 02 Module Host.kicad_sch (KiCad schematic)
At the start: 19 parts, among them J101 ICSP, J102 USB_A, SW101 SW_DIP_x08, U101 PIC18F47Q43-I/PT, U102 MCP23017_SO, U103 FT232RL

Commit message: Updates
Parts:
- renumbered C105 to C103, C109 to C104, C110 to C105, R103 to R101, R101 to R102, R102 to R103, U102 to U101, U101 to U102
Other:
- note added: "I had 10 LED bar displays and used the first 8. Discrete LEDs could be used instead. I also used a Bourns 4116R-1-331 (330 ohm) resistor pack DIP. Individual resistors could be used instead. A DIP switch is shown, but individual jumpers to ground (for bits you want to turn "On") could be used instead."
- note removed: "I had 10 LED bar displays and used the first 8. Discrete LEDs could also be used. I also used a Bourns 4116R-1-331 (330 ohm) resistor pack DIP. Individual resistors can also be used. A DIP switch is shown, but individual jumpers to ground could be used instead."
