File: Examples/Keyboard Interface/Keyboard Interface.kicad_sch (KiCad schematic)
At the start: 54 parts, among them J1 ICSP, J2 USB_A, SW1 00, SW10 13, SW11 14, SW12 15, SW13 20, SW14 21, SW15 22, SW16 23, SW17 24, SW18 25, SW19 30, SW2 01, SW20 31, SW21 32, SW22 33, SW23 34, SW24 35, SW25 40, SW26 41, SW27 42, SW28 43, SW29 44, SW3 02, SW30 45, SW4 03, SW5 04, SW6 05, SW7 10, SW8 11, SW9 12, U1 PIC18F47Q43-E/P, U2 FT232RL, U3 MCP23017_SO

Commit message: key scans
Parts:
- removed U1: PIC18F47Q43-E/P, Package_DIP:DIP-40_W16.51mm_SMDSocket_LongPads, symbol DH_MCU_Microchip:PIC18F47Q43-E/P
- added U4: PIC18F47Q43-E/PT, Package_QFP:TQFP-44_10x10mm_P0.8mm, symbol DH_MCU_Microchip:PIC18F47Q43-E/PT
Connections:
- net +5V: now also U4.28 (Vdd), U4.7 (Vdd)
- net GND: now also U4.29 (Vss), U4.6 (Vss)
- net PGC: now also U4.16 (RB6/ICSPCLK)
- net PGD: now also U4.17 (RB7/ICSPDAT)
- net SCK: now also U4.37 (RC3)
- net SDA: now also U4.42 (RC4)
- net ~{KP}: now also U4.10 (RB2)
- net ~{RESET}: now also U4.11 (RB3)

Commit message: updates
Connections:
- net LEDS is gone; now on net PWM: D9.4 (DIN)
- net PWM: now reaches U4.15 (RB5)
Changed lines of the file:
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@@
+	)
+	(bus_entry
+		(at 99.06 97.79)
+		(size 2.54 2.54)
+		(stroke
+			(width 0)
+			(type default)
+		)
 	)
 	(bus_entry
@@
 		(pts
 			(xy 115.57 64.77) (xy 116.84 64.77)
+		)
+		(stroke
+			(width 0)
+			(type default)
+		)
+	)
+	(wire
+		(pts
+			(xy 88.9 97.79) (xy 99.06 97.79)
 		)
 		(stroke
@@
 		)
 	)
-	(label "LEDS"
+	(label "PWM"
 		(at 39.37 173.99 90)
 		(effects
@@
 		(effects
 			(font
+				(size 1.27 1.27)
+			)
+			(justify left bottom)
+		)
+	)
+	(label "PWM"
+		(at 93.98 97.79 0)
+		(effects
+			(font
