File: 01 UART/UART 03 Hardware Flow Control/UART 03 Hardware Flow Control.kicad_sch (KiCad schematic)
At the start: 22 parts, among them J101 ICSP, J102 USB_A, J103 DE9_Pins, U101 PIC18F47Q43-I/PT, U102 MAX232, U103 FT232RL

Commit message: Updates
Parts:
- renumbered C103 to C101, C104 to C102, C108 to C103, C106 to C104, C107 to C105, C101 to C106, C102 to C107, C105 to C108, J103 to J102, J102 to J103, R103 to R101, R101 to R102, R102 to R103, U102 to U101, U101 to U102
Other:
- note added: "Notes: 1. Implement one or the other interface options, USB or RS-232, but not both. 2. Place C106 and C107 physically close to U102. 3. For USB interface, place C109 and C110 physically close to U103. 4. For RS-232 interface, locate C101 - C105 physically close to U101."
- note removed: "Notes: 1. Implement one or the other interface options, USB or RS-232, but not both. 2. Place C101 and C102 physically close to U101. 3. For USB interface, place C109 and C110 physically close to U103. 4. For RS-232 interface, locate C103 - C107 physically close to U102. 5. This example does not use hardware or software flow control!"
Changed lines of the file:
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@@
 		)
 	)
-	(text "Notes:\n1. Implement one or the other interface options, USB or RS-232,\n   but not both.\n2. Place C101 and C102 physically close to U101.\n3. For USB interface, place C109 and C110 physically close to U103.\n4. For RS-232 interface, locate C103 - C107 physically close to U102.\n5. This example does not use hardware or software flow control!"
+	(text "Notes:\n1. Implement one or the other interface options, USB or RS-232,\n   but not both.\n2. Place C106 and C107 physically close to U102.\n3. For USB interface, place C109 and C110 physically close to U103.\n4. For RS-232 interface, locate C101 - C105 physically close to U101."
 		(exclude_from_sim no)
 		(at 30.734 158.242 0)
@@
 		(in_pos_files yes)
 		(dnp no)
-		(property "Reference" "#PWR0117"
+		(property "Reference" "#PWR0112"
 			(at 238.76 142.24 0)
 			(hide yes)
@@
 			(project "UART 03 Hardware Flow Control"
 				(path "/d3b5dd27-4845-413f-badb-7f64f7fb8d77"
-					(reference "#PWR0117")
+					(reference "#PWR0112")
 					(unit 1)
 				)
@@
 		(in_pos_files yes)
 		(dnp no)
-		(property "Reference" "C102"
+		(property "Reference" "C107"
 			(at 122.682 54.356 0)
 			(show_name no)
@@
 			(project "UART 03 Hardware Flow Control"
 				(path "/d3b5dd27-4845-413f-badb-7f64f7fb8d77"
-					(reference "C102")
+					(reference "C107")
 					(unit 1)
 				)
@@
 		(dnp no)
 		(fields_autoplaced yes)
-		(property "Reference" "#PWR0101"
+		(property "Reference" "#PWR0102"
 			(at 41.91 33.02 0)
 			(hide yes)
@@
 			(project "UART 03 Hardware Flow Control"
 				(path "/d3b5dd27-4845-413f-badb-7f64f7fb8d77"
-					(reference "#PWR0101")
+					(reference "#PWR0102")
 					(unit 1)
 				)
@@
 		(dnp no)
 		(fields_autoplaced yes)
-		(property "Reference" "#PWR0114"
+		(property "Reference" "#PWR0115"
 			(at 223.52 156.21 0)
 			(hide yes)
@@
 			(project "UART 03 Hardware Flow Control"
 				(path "/d3b5dd27-4845-413f-badb-7f64f7fb8d77"
-					(reference "#PWR0114")
+					(reference "#PWR0115")
 					(unit 1)
 				)
@@
 		(dnp no)
 		(fields_autoplaced yes)
-		(property "Reference" "#PWR0102"
+		(property "Reference" "#PWR0103"
 			(at 41.91 52.07 0)
 			(hide yes)
@@
 			(project "UART 03 Hardware Flow Control"
 				(path "/d3b5dd27-4845-413f-badb-7f64f7fb8d77"
-					(reference "#PWR0102")
+					(reference "#PWR0103")
 					(unit 1)
 				)
@@
 		(dnp no)
 		(fields_autoplaced yes)
-		(property "Reference" "#PWR0103"
+		(property "Reference" "#PWR0104"
 			(at 106.68 55.88 0)
 			(hide yes)
@@
 			(project "UART 03 Hardware Flow Control"
 				(path "/d3b5dd27-4845-413f-badb-7f64f7fb8d77"
-					(reference "#PWR0103")
+					(reference "#PWR0104")
 					(unit 1)
 				)
@@
 		(dnp no)
 		(fields_autoplaced yes)
-		(property "Reference" "U102"
+		(property "Reference" "U101"
 			(at 183.7533 25.4 0)
 			(show_name no)
@@
 			(project "UART 03 Hardware Flow Control"
 				(path "/d3b5dd27-4845-413f-badb-7f64f7fb8d77"
-					(reference "U102")
+					(reference "U101")
 					(unit 1)
 				)
@@
 		(dnp no)
 		(fields_autoplaced yes)
-		(property "Reference" "#PWR0108"
+		(property "Reference" "#PWR0117"
 			(at 177.8 167.64 0)
 			(hide yes)
@@
 			(project "UART 03 Hardware Flow Control"
 				(path "/d3b5dd27-4845-413f-badb-7f64f7fb8d77"
-					(reference "#PWR0108")
+					(reference "#PWR0117")
 					(unit 1)
 				)
@@
 		(dnp no)
 		(fields_autoplaced yes)
-		(property "Reference" "#PWR0107"
+		(property "Reference" "#PWR0113"
 			(at 140.97 140.97 0)
 			(hide yes)
@@
 			(project "UART 03 Hardware Flow Control"
 				(path "/d3b5dd27-4845-413f-badb-7f64f7fb8d77"
-					(reference "#PWR0107")
+					(reference "#PWR0113")
 					(unit 1)
 				)
@@
 		(dnp no)
 		(fields_autoplaced yes)
-		(property "Reference" "R103"
+		(property "Reference" "R101"
 			(at 226.06 130.8099 0)
 			(show_name no)
@@
 			(project "UART 03 Hardware Flow Control"
 				(path "/d3b5dd27-4845-413f-badb-7f64f7fb8d77"
-					(reference "R103")
+					(reference "R101")
 					(unit 1)
 				)
@@
 		(in_pos_files yes)
 		(dnp no)
-		(property "Reference" "C101"
+		(property "Reference" "C106"
 			(at 114.808 54.864 0)
 			(show_name no)
@@
 			(project "UART 03 Hardware Flow Control"
 				(path "/d3b5dd27-4845-413f-badb-7f64f7fb8d77"
-					(reference "C101")
+					(reference "C106")
 					(unit 1)
 				)
@@
 		(in_pos_files yes)
 		(dnp no)
-		(property "Reference" "C104"
+		(property "Reference" "C102"
 			(at 206.248 33.02 0)
 			(show_name no)
@@
 			(project "UART 03 Hardware Flow Control"
 				(path "/d3b5dd27-4845-413f-badb-7f64f7fb8d77"
-					(reference "C104")
+					(reference "C102")
 					(unit 1)
 				)
@@
 		(in_pos_files yes)
 		(dnp no)
-		(property "Reference" "R101"
+		(property "Reference" "R102"
 			(at 148.082 135.636 90)
 			(show_name no)
@@
 			(project "UART 03 Hardware Flow Control"
 				(path "/d3b5dd27-4845-413f-badb-7f64f7fb8d77"
-					(reference "R101")
+					(reference "R102")
 					(unit 1)
 				)
@@
 		(in_pos_files yes)
 		(dnp no)
-		(property "Reference" "#PWR0115"
+		(property "Reference" "#PWR0114"
 			(at 234.95 149.86 0)
 			(hide yes)
@@
 			(project "UART 03 Hardware Flow Control"
 				(path "/d3b5dd27-4845-413f-badb-7f64f7fb8d77"
-					(reference "#PWR0115")
+					(reference "#PWR0114")
 					(unit 1)
 				)
@@
 		(dnp no)
 		(fields_autoplaced yes)
-		(property "Reference" "#PWR0110"
+		(property "Reference" "#PWR0101"
 			(at 181.61 25.4 0)
 			(hide yes)
@@
 			(project "UART 03 Hardware Flow Control"
 				(path "/d3b5dd27-4845-413f-badb-7f64f7fb8d77"
-					(reference "#PWR0110")
+					(reference "#PWR0101")
 					(unit 1)
 				)
@@
 		(in_pos_files yes)
 		(dnp no)
-		(property "Reference" "J102"
+		(property "Reference" "J103"
 			(at 238.76 109.22 0)
 			(show_name no)
@@
 			(project "UART 03 Hardware Flow Control"
 				(path "/d3b5dd27-4845-413f-badb-7f64f7fb8d77"
-					(reference "J102")
+					(reference "J103")
 					(unit 1)
 				)
@@
 		(in_pos_files yes)
 		(dnp no)
-		(property "Reference" "C108"
+		(property "Reference" "C103"
 			(at 218.948 33.274 0)
 			(show_name no)
@@
 			(project "UART 03 Hardware Flow Control"
 				(path "/d3b5dd27-4845-413f-badb-7f64f7fb8d77"
-					(reference "C108")
+					(reference "C103")
 					(unit 1)
 				)
@@
 		(dnp no)
 		(fields_autoplaced yes)
-		(property "Reference" "U101"
+		(property "Reference" "U102"
 			(at 82.55 46.99 0)
 			(show_name no)
@@
 			(project "UART 03 Hardware Flow Control"
 				(path "/d3b5dd27-4845-413f-badb-7f64f7fb8d77"
-					(reference "U101")
+					(reference "U102")
 					(unit 1)
 				)
@@
 		(dnp no)
 		(fields_autoplaced yes)
-		(property "Reference" "#PWR0104"
+		(property "Reference" "#PWR0111"
 			(at 106.68 134.62 0)
 			(hide yes)
@@
 			(project "UART 03 Hardware Flow Control"
 				(path "/d3b5dd27-4845-413f-badb-7f64f7fb8d77"
-					(reference "#PWR0104")
+					(reference "#PWR0111")
 					(unit 1)
 				)
@@
 		(in_pos_files yes)
 		(dnp no)
-		(property "Reference" "#PWR0111"
+		(property "Reference" "#PWR0108"
 			(at 181.61 93.98 0)
 			(hide yes)
@@
 			(project "UART 03 Hardware Flow Control"
 				(path "/d3b5dd27-4845-413f-badb-7f64f7fb8d77"
-					(reference "#PWR0111")
+					(reference "#PWR0108")
 					(unit 1)
 				)
@@
 		(dnp no)
 		(fields_autoplaced yes)
-		(property "Reference" "C103"
+		(property "Reference" "C101"
 			(at 156.21 35.1281 0)
 			(show_name no)
@@
 			(project "UART 03 Hardware Flow Control"
 				(path "/d3b5dd27-4845-413f-badb-7f64f7fb8d77"
-					(reference "C103")
+					(reference "C101")
 					(unit 1)
 				)
@@
 		(in_pos_files yes)
 		(dnp no)
-		(property "Reference" "C106"
+		(property "Reference" "C104"
 			(at 207.772 42.418 90)
 			(show_name no)
@@
 			(project "UART 03 Hardware Flow Control"
 				(path "/d3b5dd27-4845-413f-badb-7f64f7fb8d77"
-					(reference "C106")
+					(reference "C104")
 					(unit 1)
 				)
@@
 		(in_pos_files yes)
 		(dnp no)
-		(property "Reference" "C107"
+		(property "Reference" "C105"
 			(at 207.518 49.784 90)
 			(show_name no)
@@
 			(project "UART 03 Hardware Flow Control"
 				(path "/d3b5dd27-4845-413f-badb-7f64f7fb8d77"
-					(reference "C107")
+					(reference "C105")
 					(unit 1)
 				)
@@
 		(in_pos_files yes)
 		(dnp no)
-		(property "Reference" "R102"
+		(property "Reference" "R103"
 			(at 147.828 144.78 90)
 			(show_name no)
@@
 			(project "UART 03 Hardware Flow Control"
 				(path "/d3b5dd27-4845-413f-badb-7f64f7fb8d77"
-					(reference "R102")
+					(reference "R103")
 					(unit 1)
 				)
@@
 		(dnp no)
 		(fields_autoplaced yes)
-		(property "Reference" "#PWR0113"
+		(property "Reference" "#PWR0110"
 			(at 219.71 121.92 0)
 			(hide yes)
@@
 			(project "UART 03 Hardware Flow Control"
 				(path "/d3b5dd27-4845-413f-badb-7f64f7fb8d77"
-					(reference "#PWR0113")
+					(reference "#PWR0110")
 					(unit 1)
 				)
@@
 		(dnp no)
 		(fields_autoplaced yes)
-		(property "Reference" "C105"
+		(property "Reference" "C108"
 			(at 211.074 106.68 90)
 			(show_name no)
@@
 			(project "UART 03 Hardware Flow Control"
 				(path "/d3b5dd27-4845-413f-badb-7f64f7fb8d77"
-					(reference "C105")
+					(reference "C108")
 					(unit 1)
 				)
@@
 		(in_pos_files yes)
 		(dnp no)
-		(property "Reference" "J103"
+		(property "Reference" "J102"
 			(at 245.11 67.3101 0)
 			(show_name no)
@@
 			(project "UART 03 Hardware Flow Control"
 				(path "/d3b5dd27-4845-413f-badb-7f64f7fb8d77"
-					(reference "J103")
+					(reference "J102")
 					(unit 1)
 				)
@@
 		(dnp no)
 		(fields_autoplaced yes)
-		(property "Reference" "#PWR0112"
+		(property "Reference" "#PWR0107"
 			(at 218.44 87.63 0)
 			(hide yes)
@@
 			(project "UART 03 Hardware Flow Control"
 				(path "/d3b5dd27-4845-413f-badb-7f64f7fb8d77"
-					(reference "#PWR0112")
+					(reference "#PWR0107")
 					(unit 1)
 				)
