File: 01 UART/UART 04 Software Flow Control/UART 04 Software Flow Control.kicad_sch (KiCad schematic)
At the start: 22 parts, among them J101 ICSP, J102 USB_A, J103 DE9_Pins, U101 PIC18F47Q43-I/PT, U102 MAX232, U103 FT232RL

Commit message: Updates
Parts:
- renumbered C103 to C101, C104 to C102, C108 to C103, C106 to C104, C107 to C105, C101 to C106, C102 to C107, C105 to C108, J103 to J102, J102 to J103, R103 to R101, R101 to R102, R102 to R103, U102 to U101, U101 to U102
Other:
- note added: "Notes: 1. Implement one or the other interface options, USB or RS-232, but not both. 2. Place C106 and C107 physically close to U102. 3. For USB interface, place C109 and C110 physically close to U103. 4. For RS-232 interface, locate C101 - C105 physically close to U101."
- note removed: "Notes: 1. Implement one or the other interface options, USB or RS-232, but not both. 2. Place C101 and C102 physically close to U101. 3. For USB interface, place C109 and C110 physically close to U103. 4. For RS-232 interface, locate C103 - C107 physically close to U102. 5. This example does not use hardware or software flow control!"
