File: 02 IOC/IOC 01 Single/IOC_Single.kicad_sch (KiCad schematic)
At the start: 17 parts, among them J1 ICSP, J102 USB_A, SW1 SW_DIP_x08, U1 PIC18F47Q43-I/PT, U103 FT232RL

Commit message: Updates
Parts:
- renumbered BAR1 to BAR101, C1 to C101, C105 to C102, C109 to C103, C110 to C104, J1 to J101, R103 to R101, R101 to R102, R102 to R103, RN1 to RN101, SW1 to SW101, U1 to U101, U103 to U102
Changed lines of the file:
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@@
 		(in_pos_files yes)
 		(dnp no)
-		(property "Reference" "J1"
+		(property "Reference" "J101"
 			(at 26.67 29.2099 0)
 			(show_name no)
@@
 			(project "IOC_Single"
 				(path "/a268f71e-0835-4511-aa86-9e5be2256047"
-					(reference "J1")
+					(reference "J101")
 					(unit 1)
 				)
@@
 		(in_pos_files yes)
 		(dnp no)
-		(property "Reference" "#PWR0117"
+		(property "Reference" "#PWR0111"
 			(at 242.57 140.97 0)
 			(hide yes)
@@
 			(project "IOC_Single"
 				(path "/a268f71e-0835-4511-aa86-9e5be2256047"
-					(reference "#PWR0117")
+					(reference "#PWR0111")
 					(unit 1)
 				)
@@
 		(in_pos_files yes)
 		(dnp no)
-		(property "Reference" "#PWR0116"
+		(property "Reference" "#PWR0115"
 			(at 238.76 163.83 0)
 			(hide yes)
@@
 			(project "IOC_Single"
 				(path "/a268f71e-0835-4511-aa86-9e5be2256047"
-					(reference "#PWR0116")
+					(reference "#PWR0115")
 					(unit 1)
 				)
@@
 		(in_pos_files yes)
 		(dnp no)
-		(property "Reference" "#PWR08"
+		(property "Reference" "#PWR0105"
 			(at 116.84 55.88 0)
 			(hide yes)
@@
 			(project "IOC_Single"
 				(path "/a268f71e-0835-4511-aa86-9e5be2256047"
-					(reference "#PWR08")
+					(reference "#PWR0105")
 					(unit 1)
 				)
@@
 		(dnp no)
 		(fields_autoplaced yes)
-		(property "Reference" "SW1"
+		(property "Reference" "SW101"
 			(at 38.1 88.9 0)
 			(show_name no)
@@
 			(project "IOC_Single"
 				(path "/a268f71e-0835-4511-aa86-9e5be2256047"
-					(reference "SW1")
+					(reference "SW101")
 					(unit 1)
 				)
@@
 		(dnp no)
 		(fields_autoplaced yes)
-		(property "Reference" "#PWR0108"
+		(property "Reference" "#PWR0116"
 			(at 181.61 166.37 0)
 			(hide yes)
@@
 			(project "IOC_Single"
 				(path "/a268f71e-0835-4511-aa86-9e5be2256047"
-					(reference "#PWR0108")
+					(reference "#PWR0116")
 					(unit 1)
 				)
@@
 		(in_pos_files yes)
 		(dnp no)
-		(property "Reference" "#PWR0109"
+		(property "Reference" "#PWR0107"
 			(at 184.15 105.41 0)
 			(hide yes)
@@
 			(project "IOC_Single"
 				(path "/a268f71e-0835-4511-aa86-9e5be2256047"
-					(reference "#PWR0109")
+					(reference "#PWR0107")
 					(unit 1)
 				)
@@
 		(dnp no)
 		(fields_autoplaced yes)
-		(property "Reference" "#PWR0107"
+		(property "Reference" "#PWR0112"
 			(at 144.78 139.7 0)
 			(hide yes)
@@
 			(project "IOC_Single"
 				(path "/a268f71e-0835-4511-aa86-9e5be2256047"
-					(reference "#PWR0107")
+					(reference "#PWR0112")
 					(unit 1)
 				)
@@
 		(dnp no)
 		(fields_autoplaced yes)
-		(property "Reference" "R103"
+		(property "Reference" "R101"
 			(at 229.87 129.5399 0)
 			(show_name no)
@@
 			(project "IOC_Single"
 				(path "/a268f71e-0835-4511-aa86-9e5be2256047"
-					(reference "R103")
+					(reference "R101")
 					(unit 1)
 				)
@@
 		(dnp no)
 		(fields_autoplaced yes)
-		(property "Reference" "#PWR07"
+		(property "Reference" "#PWR0104"
 			(at 116.84 41.91 0)
 			(hide yes)
@@
 			(project "IOC_Single"
 				(path "/a268f71e-0835-4511-aa86-9e5be2256047"
-					(reference "#PWR07")
+					(reference "#PWR0104")
 					(unit 1)
 				)
@@
 		(in_pos_files yes)
 		(dnp no)
-		(property "Reference" "BAR1"
+		(property "Reference" "BAR101"
 			(at 123.19 98.298 0)
 			(show_name no)
@@
 			(project "IOC_Single"
 				(path "/a268f71e-0835-4511-aa86-9e5be2256047"
-					(reference "BAR1")
+					(reference "BAR101")
 					(unit 1)
 				)
@@
 		(in_pos_files yes)
 		(dnp no)
-		(property "Reference" "#PWR03"
+		(property "Reference" "#PWR0109"
 			(at 27.94 121.92 0)
 			(hide yes)
@@
 			(project "IOC_Single"
 				(path "/a268f71e-0835-4511-aa86-9e5be2256047"
-					(reference "#PWR03")
+					(reference "#PWR0109")
 					(unit 1)
 				)
@@
 		(in_pos_files yes)
 		(dnp no)
-		(property "Reference" "R101"
+		(property "Reference" "R102"
 			(at 151.892 134.366 90)
 			(show_name no)
@@
 			(project "IOC_Single"
 				(path "/a268f71e-0835-4511-aa86-9e5be2256047"
-					(reference "R101")
+					(reference "R102")
 					(unit 1)
 				)
@@
 		(dnp no)
 		(fields_autoplaced yes)
-		(property "Reference" "#PWR06"
+		(property "Reference" "#PWR0102"
 			(at 35.56 44.45 0)
 			(hide yes)
@@
 			(project "IOC_Single"
 				(path "/a268f71e-0835-4511-aa86-9e5be2256047"
-					(reference "#PWR06")
+					(reference "#PWR0102")
 					(unit 1)
 				)
@@
 		(in_pos_files yes)
 		(dnp no)
-		(property "Reference" "#PWR0115"
+		(property "Reference" "#PWR0113"
 			(at 238.76 148.59 0)
 			(hide yes)
@@
 			(project "IOC_Single"
 				(path "/a268f71e-0835-4511-aa86-9e5be2256047"
-					(reference "#PWR0115")
+					(reference "#PWR0113")
 					(unit 1)
 				)
@@
 		(dnp no)
 		(fields_autoplaced yes)
-		(property "Reference" "#PWR04"
+		(property "Reference" "#PWR0106"
 			(at 154.94 68.58 0)
 			(hide yes)
@@
 			(project "IOC_Single"
 				(path "/a268f71e-0835-4511-aa86-9e5be2256047"
-					(reference "#PWR04")
+					(reference "#PWR0106")
 					(unit 1)
 				)
@@
 		(dnp no)
 		(fields_autoplaced yes)
-		(property "Reference" "#PWR01"
+		(property "Reference" "#PWR0103"
 			(at 104.14 41.91 0)
 			(hide yes)
@@
 			(project "IOC_Single"
 				(path "/a268f71e-0835-4511-aa86-9e5be2256047"
-					(reference "#PWR01")
+					(reference "#PWR0103")
 					(unit 1)
 				)
@@
 		(dnp no)
 		(fields_autoplaced yes)
-		(property "Reference" "#PWR02"
+		(property "Reference" "#PWR0110"
 			(at 104.14 124.46 0)
 			(hide yes)
@@
 			(project "IOC_Single"
 				(path "/a268f71e-0835-4511-aa86-9e5be2256047"
-					(reference "#PWR02")
+					(reference "#PWR0110")
 					(unit 1)
 				)
@@
 		(dnp no)
 		(fields_autoplaced yes)
-		(property "Reference" "U1"
+		(property "Reference" "U101"
 			(at 78.74 35.56 0)
 			(show_name no)
@@
 			(project "IOC_Single"
 				(path "/a268f71e-0835-4511-aa86-9e5be2256047"
-					(reference "U1")
+					(reference "U101")
 					(unit 1)
 				)
@@
 		(dnp no)
 		(fields_autoplaced yes)
-		(property "Reference" "#PWR05"
+		(property "Reference" "#PWR0101"
 			(at 35.56 26.67 0)
 			(hide yes)
@@
 			(project "IOC_Single"
 				(path "/a268f71e-0835-4511-aa86-9e5be2256047"
-					(reference "#PWR05")
+					(reference "#PWR0101")
 					(unit 1)
 				)
@@
 		(dnp no)
 		(fields_autoplaced yes)
-		(property "Reference" "RN1"
+		(property "Reference" "RN101"
 			(at 144.78 64.77 90)
 			(show_name no)
@@
 			(project "IOC_Single"
 				(path "/a268f71e-0835-4511-aa86-9e5be2256047"
-					(reference "RN1")
+					(reference "RN101")
 					(unit 1)
 				)
@@
 		(in_pos_files yes)
 		(dnp no)
-		(property "Reference" "C110"
+		(property "Reference" "C104"
 			(at 247.142 147.066 0)
 			(show_name no)
@@
 			(project "IOC_Single"
 				(path "/a268f71e-0835-4511-aa86-9e5be2256047"
-					(reference "C110")
+					(reference "C104")
 					(unit 1)
 				)
@@
 		(in_pos_files yes)
 		(dnp no)
-		(property "Reference" "C109"
+		(property "Reference" "C103"
 			(at 239.268 147.574 0)
 			(show_name no)
@@
 			(project "IOC_Single"
 				(path "/a268f71e-0835-4511-aa86-9e5be2256047"
-					(reference "C109")
+					(reference "C103")
 					(unit 1)
 				)
@@
 		(in_pos_files yes)
 		(dnp no)
-		(property "Reference" "U103"
+		(property "Reference" "U102"
 			(at 182.0067 104.14 0)
 			(show_name no)
@@
 			(project "IOC_Single"
 				(path "/a268f71e-0835-4511-aa86-9e5be2256047"
-					(reference "U103")
+					(reference "U102")
 					(unit 1)
 				)
@@
 		(in_pos_files yes)
 		(dnp no)
-		(property "Reference" "R102"
+		(property "Reference" "R103"
 			(at 151.638 143.51 90)
 			(show_name no)
@@
 			(project "IOC_Single"
 				(path "/a268f71e-0835-4511-aa86-9e5be2256047"
-					(reference "R102")
+					(reference "R103")
 					(unit 1)
 				)
@@
 		(dnp no)
 		(fields_autoplaced yes)
-		(property "Reference" "C1"
+		(property "Reference" "C101"
 			(at 120.65 42.1639 0)
 			(show_name no)
@@
 			(project "IOC_Single"
 				(path "/a268f71e-0835-4511-aa86-9e5be2256047"
-					(reference "C1")
+					(reference "C101")
 					(unit 1)
 				)
@@
 		(dnp no)
 		(fields_autoplaced yes)
-		(property "Reference" "#PWR0113"
+		(property "Reference" "#PWR0108"
 			(at 223.52 120.65 0)
 			(hide yes)
@@
 			(project "IOC_Single"
 				(path "/a268f71e-0835-4511-aa86-9e5be2256047"
-					(reference "#PWR0113")
+					(reference "#PWR0108")
 					(unit 1)
 				)
@@
 		(dnp no)
 		(fields_autoplaced yes)
-		(property "Reference" "C105"
+		(property "Reference" "C102"
 			(at 214.884 105.41 90)
 			(show_name no)
@@
 			(project "IOC_Single"
 				(path "/a268f71e-0835-4511-aa86-9e5be2256047"
-					(reference "C105")
-					(unit 1)
-				)
+					(reference "C102")
+					(unit 1)
+				)
