File: 02 IOC/IOC 02 Vectored/IOC_Vectored.kicad_sch (KiCad schematic)
At the start: 17 parts, among them J1 ICSP, J102 USB_A, SW1 SW_DIP_x08, U1 PIC18F47Q43-I/PT, U103 FT232RL

Commit message: Updates
Parts:
- renumbered BAR1 to BAR101, C1 to C101, C105 to C102, C109 to C103, C110 to C104, J1 to J101, R103 to R101, R101 to R102, R102 to R103, RN1 to RN101, SW1 to SW101, U1 to U101, U103 to U102
