File: 03 I2C/I2C 01 Bit Bang Host/I2C 01 Bit Bang Master.kicad_sch (KiCad schematic)
At the start: 21 parts, among them J101 ICSP, J102 USB_A, SW101 SW_DIP_x08, U101 PIC18F47Q43-I/PT, U102 MCP23017_SO, U103 FT232RL

Commit message: Updates
Parts:
- renumbered C105 to C103, C109 to C104, C110 to C105, R105 to R101, R106 to R102, R101 to R104, R102 to R105, R104 to R106, U102 to U101, U101 to U102
Connections:
- net ~{RESET}: now also U102.11 (RB3); no longer J101.1 (Pin_1), U102.18 (~{MCLR}/Vpp/RE3)
- new net: J101.1 (Pin_1), U102.18 (~{MCLR}/Vpp/RE3)
- no-connect marks 42 -> 41
