File: 13 PWM/PWM 02 Fan Control/_autosave-Fan Control.kicad_sch (KiCad schematic)
At the start: 20 parts, among them J1 Fan, J101 ICSP, J102 USB_A, J2 Fan, M1 Fan_4pin, U101 PIC18F47Q43-I/PT, U102 FT232RL

Commit message: Added PWM fan control
Parts:
- removed R107: 10K, symbol Device:R_US
Other:
- note added: "Configured as open drain output, the fan will pull up this pin."
- note removed: "Configured as open drain."
Changed lines of the file:
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@@
 	(text "Use pull-up on pin."
 		(exclude_from_sim no)
-		(at 112.776 141.478 0)
+		(at 108.966 141.478 0)
 		(effects
 			(font
@@
 		)
 	)
-	(text "Configured as open drain. "
+	(text "Configured as open drain output,\nthe fan will pull up this pin. "
 		(exclude_from_sim no)
-		(at 112.776 146.558 0)
+		(at 109.22 147.828 0)
 		(effects
 			(font
@@
 	)
 	(junction
-		(at 160.02 144.78)
-		(diameter 0)
-		(color 0 0 0 0)
-	)
-	(junction
 		(at 134.62 208.28)
 		(diameter 0)
@@
 	(wire
 		(pts
-			(xy 160.02 129.54) (xy 160.02 132.08)
-		)
-		(stroke
-			(width 0)
-			(type default)
-		)
-	)
-	(wire
-		(pts
 			(xy 135.89 49.53) (xy 135.89 50.8)
 		)
@@
 	(wire
 		(pts
-			(xy 160.02 139.7) (xy 160.02 144.78)
-		)
-		(stroke
-			(width 0)
-			(type default)
-		)
-	)
-	(wire
-		(pts
 			(xy 102.87 175.26) (xy 130.81 175.26)
 		)
@@
 	(wire
 		(pts
-			(xy 60.96 144.78) (xy 160.02 144.78)
+			(xy 60.96 144.78) (xy 172.72 144.78)
 		)
 		(stroke
@@
 		(pts
 			(xy 87.63 210.82) (xy 85.09 210.82)
-		)
-		(stroke
-			(width 0)
-			(type default)
-		)
-	)
-	(wire
-		(pts
-			(xy 160.02 144.78) (xy 172.72 144.78)
 		)
 		(stroke
@@
 	)
 	(symbol
-		(lib_id "power:+5V")
-		(at 160.02 129.54 0)
-		(unit 1)
-		(body_style 1)
-		(exclude_from_sim no)
-		(in_bom yes)
-		(on_board yes)
-		(in_pos_files yes)
-		(dnp no)
-		(property "Reference" "#PWR0109"
-			(at 160.02 133.35 0)
-			(hide yes)
-			(show_name no)
-			(do_not_autoplace no)
-			(effects
-				(font
-					(size 1.27 1.27)
-				)
-			)
-		)
-		(property "Value" "+5V"
-			(at 160.274 125.984 0)
-			(show_name no)
-			(do_not_autoplace no)
-			(effects
-				(font
-					(size 1.27 1.27)
-				)
-			)
-		)
-		(property "Footprint" ""
-			(at 160.02 129.54 0)
-			(hide yes)
-			(show_name no)
-			(do_not_autoplace no)
-			(effects
-				(font
-					(size 1.27 1.27)
-				)
-			)
-		)
-		(property "Datasheet" ""
-			(at 160.02 129.54 0)
-			(hide yes)
-			(show_name no)
-			(do_not_autoplace no)
-			(effects
-				(font
-					(size 1.27 1.27)
-				)
-			)
-		)
-		(property "Description" "Power symbol creates a global label with name \"+5V\""
-			(at 160.02 129.54 0)
-			(hide yes)
-			(show_name no)
-			(do_not_autoplace no)
-			(effects
-				(font
-					(size 1.27 1.27)
-				)
-			)
-		)
-		(pin "1"
-		)
-		(instances
-			(project "Fan Control"
-				(path "/badc57c4-ca21-4b51-becd-f0bffd352e4b"
-					(reference "#PWR0109")
-					(unit 1)
-				)
-			)
-		)
-	)
-	(symbol
 		(lib_id "power:GND")
 		(at 135.89 60.96 0)
@@
 					(unit 1)
 				)
-			)
-		)
-	)
-	(symbol
-		(lib_id "Device:R_US")
-		(at 160.02 135.89 0)
-		(unit 1)
-		(body_style 1)
-		(exclude_from_sim no)
-		(in_bom yes)
-		(on_board yes)
-		(in_pos_files yes)
-		(dnp no)
-		(fields_autoplaced yes)
-		(property "Reference" "R107"
-			(at 162.56 134.6199 0)
-			(show_name no)
-			(do_not_autoplace no)
-			(effects
-				(font
-					(size 1.27 1.27)
-				)
-				(justify left)
-			)
-		)
-		(property "Value" "10K"
-			(at 162.56 137.1599 0)
-			(show_name no)
-			(do_not_autoplace no)
-			(effects
-				(font
-					(size 1.27 1.27)
-				)
-				(justify left)
-			)
-		)
-		(property "Footprint" ""
-			(at 161.036 136.144 90)
-			(hide yes)
-			(show_name no)
-			(do_not_autoplace no)
-			(effects
-				(font
-					(size 1.27 1.27)
-				)
-			)
-		)
-		(property "Datasheet" ""
-			(at 160.02 135.89 0)
-			(hide yes)
-			(show_name no)
-			(do_not_autoplace no)
-			(effects
-				(font
-					(size 1.27 1.27)
-				)
-			)
-		)
-		(property "Description" "Resistor, US symbol"
-			(at 160.02 135.89 0)
-			(hide yes)
-			(show_name no)
-			(do_not_autoplace no)
-			(effects
-				(font
-					(size 1.27 1.27)
-				)
-			)
-		)
-		(pin "2"
-		)
-		(pin "1"
-		)
-		(instances
-			(project "Fan Control"
-				(path "/badc57c4-ca21-4b51-becd-f0bffd352e4b"
-					(reference "R107")
-					(unit 1)
-				)
