File: 13 PWM/PWM 02 Fan Control/Fan Control.kicad_sch (KiCad schematic)
At the start: 20 parts, among them J1 Fan, J101 ICSP, J102 USB_A, J2 Fan, M1 Fan_4pin, U101 PIC18F47Q43-I/PT, U102 FT232RL

Commit message: update
Parts:
- removed R107: 10K, symbol Device:R_US
Connections:
- net at J2.3 (Pin_3): no longer M1.3 (Tacho)
- net at J2.4 (Pin_4): no longer M1.4 (PWM)
Other:
- note added: "Configured as open drain output, the fan will pull up this pin."
- note removed: "Configured as open drain."
- moved on the sheet: D1, J1, J2, R106

Commit message: after code review
Parts:
- removed J1, J2: Fan, symbol Connector_Generic:Conn_01x04
Connections:
- net +12V: now also M1.2 (+)
- net GND: now also M1.1 (-), U102.18 (GND)
- net PWM: now also U101.36 (RC2); no longer U101.32 (RC0)
- net TACH: now also U101.32 (RC0); no longer U101.36 (RC2)
- net at R106.2: now also M1.4 (PWM)
- net at D1.1 (K): now also M1.3 (Tacho)
- no-connect marks 11 -> 40
Other:
- moved on the sheet: D1, M1, R106

Commit message: updated
Parts:
- removed D1: 1N4148, Diode_THT:D_DO-35_SOD27_P7.62mm_Horizontal, symbol Diode:1N4148
- added C5, C6: 0.1uF, symbol Device:C_US
- added D3, D4, D5, D6: 1N5819, Diode_THT:D_DO-41_SOD81_P10.16mm_Horizontal, symbol Diode:1N5819
- added R5: 10K, symbol Device:R_US
- added R6: 47, symbol Device:R_US
- R7: renamed from R106; value 1K -> 47
- renumbered C102 to C1, C103 to C2, C101 to C3, C104 to C4, D101 to D1, D102 to D2, J101 to J1, J102 to J2, R102 to R1, R103 to R2, R101 to R3, R104 to R4, U102 to U1, U101 to U2
Connections:
- net +5V: now also C5.1, C6.1, D3.1 (K), D5.1 (K), R5.2
- net GND: now also C5.2, C6.2, D4.2 (A), D6.2 (A)
- net PWM: now also D5.2 (A), D6.1 (K)
- net TACH: now also D3.2 (A), D4.1 (K), R6.1
- net at J1.1 (Pin_1), U2.18 (~{MCLR}/Vpp/RE3): now also R5.1
- net at M1.3 (Tacho): now also R6.2
Other:
- note added: "Between pin 20 and 21 of U1"
- note added: "Between pin 28 and 29 of U2"
- note added: "Between pin 6 and 7 of U2"
- company: (none) -> Dewayne Hafenstein
- title: (none) -> PWM 02 Fan Control
- moved on the sheet: C1, C2, C3, C4, D1, D2, J1, J2, M1, R1, R2, R3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
